File: ECAD/PCBs for Sim/IFEI/IFEI.sch (KiCad schematic (older format))
At the start: 11 parts, among them J1 Conn_01x05_Male, SW1 mode, SW2 qty, SW3 up, SW4 down, SW5 zone, SW6 ET

Commit message: Updated IFEI PCB to 2x4 pin header
#39 Updated IFEI PCB to 2x4 pin header.

Requires manufacturing files.
Parts:
- J1: value Conn_01x05_Male -> Conn_02x04_Male; footprint Pin_Headers:Pin_Header_Angled_1x05_Pitch2.54mm -> Connector_PinHeader_2.54mm:PinHeader_2x04_P2.54mm_Horizontal; symbol Connector:Conn_01x05_Male -> Connector_Generic:Conn_02x04_Odd_Even
Connections:
- net labels added: A, B, C, D, E, F, GND
- net labels removed: a, b, c, d, e
- wire segments 0 -> 18
Other:
- moved on the sheet: MK1, MK2, MK3, MK4, SW1, SW2, SW3, SW4, SW5, SW6
