File: ECAD/lib/templates/ABSIS_Nano_2.0_Template/ABSIS_Nano_2.0_Template.sch (KiCad schematic (older format))
At the start: 17 parts, among them J1 BUS IN, J2 BUS OUT, P1 Digital, P2 Analog, P3 CONN_01X01, P4 CONN_01X01, P5 CONN_01X01, P6 CONN_01X01, U1 MAX487EESA+T

Commit message: Small tweaks
Cosmetic tweaks to Master Schematic
Updated Nano template with correct J1/J2 schematic pinouts.
Parts:
- J1, J2: symbol Connector_Generic:Conn_02x03_Counter_Clockwise -> Connector_Generic:Conn_02x03_Top_Bottom
Changed lines of the file:
@@
 EESchema Schematic File Version 4
-LIBS:ABSIS_Nano-cache
 EELAYER 30 0
 EELAYER END
@@
 $EndComp
 $Comp
-L Connector_Generic:Conn_02x03_Counter_Clockwise J1
+L Connector_Generic:Conn_02x03_Top_Bottom J1
 U 1 1 5FA7581B
 P 14550 4200
@@
 Text Label 15450 5500 0    50   ~ 0
 BUS-A
-Text Label 14850 4300 0    50   ~ 0
+Text Label 14850 4100 0    50   ~ 0
 BUS-A
 Text Label 14850 4200 0    50   ~ 0
@@
 L power:GND #PWR0106
 U 1 1 5FA794C6
-P 14900 4050
-F 0 "#PWR0106" H 14900 3800 50  0001 C CNN
-F 1 "GND" H 14900 3900 50  0000 C CNN
-F 2 "" H 14900 4050 50  0000 C CNN
-F 3 "" H 14900 4050 50  0000 C CNN
-	1    14900 4050
-	0    -1   -1   0
-$EndComp
-Wire Wire Line
-	14850 4100 14900 4100
-Wire Wire Line
-	14900 4100 14900 4050
+P 14850 4300
+F 0 "#PWR0106" H 14850 4050 50  0001 C CNN
+F 1 "GND" H 14850 4150 50  0000 C CNN
+F 2 "" H 14850 4300 50  0000 C CNN
+F 3 "" H 14850 4300 50  0000 C CNN
+	1    14850 4300
+	0    -1   -1   0
+$EndComp
 Text Label 14350 4100 2    50   ~ 0
 +12V_SUPPLY
@@
 3(**)
 $Comp
-L Connector_Generic:Conn_02x03_Counter_Clockwise J2
+L Connector_Generic:Conn_02x03_Top_Bottom J2
 U 1 1 5FA822FB
 P 15900 4200
@@
 	1    0    0    -1
 $EndComp
-Text Label 16200 4300 0    50   ~ 0
+Text Label 16200 4100 0    50   ~ 0
 BUS-A
 Text Label 16200 4200 0    50   ~ 0
@@
 L power:GND #PWR0109
 U 1 1 5FA82307
-P 16250 4050
-F 0 "#PWR0109" H 16250 3800 50  0001 C CNN
-F 1 "GND" H 16250 3900 50  0000 C CNN
-F 2 "" H 16250 4050 50  0000 C CNN
-F 3 "" H 16250 4050 50  0000 C CNN
-	1    16250 4050
-	0    -1   -1   0
-$EndComp
-Wire Wire Line
-	16200 4100 16250 4100
-Wire Wire Line
-	16250 4100 16250 4050
+P 16200 4300
+F 0 "#PWR0109" H 16200 4050 50  0001 C CNN
+F 1 "GND" H 16200 4150 50  0000 C CNN
+F 2 "" H 16200 4300 50  0000 C CNN
+F 3 "" H 16200 4300 50  0000 C CNN
+	1    16200 4300
+	0    -1   -1   0
+$EndComp
 Text Label 15700 4100 2    50   ~ 0
 +12V_SUPPLY
