File: ECAD/PCBs/ABSIS/ABSIS_ATX_PSU_Board/ATX_PSU_Board/ATX_PSU_Board.sch (KiCad schematic (older format))
At the start: 22 parts, among them J1 Power Swtich, J10 MEGA BUS POWER, J2 ATX-24, J3 ABSIS BACKLIGHT PWR, J4 MEGA BUS POWER, J5 MEGA BUS POWER, J6 MEGA BUS POWER, J7 MEGA BUS POWER, J8 MEGA BUS POWER, J9 MEGA BUS POWER

Commit message: Added Gerber and Production Files
Parts:
- D4: Category Optoelectronics -> (none); Family LED Indication - Discrete -> (none); Manufacture PN FC-DA1608UGK-520D10 -> (none)
Changed lines of the file:
@@
 Wire Wire Line
 	9350 1200 9500 1200
-Wire Wire Line
-	9800 1200 9850 1200
 $Comp
 L Device:R R2
@@
 Text Notes 1550 1000 0    50   ~ 0
 Power Connectors
-Connection ~ 9850 1200
-Wire Wire Line
-	9850 1200 9950 1200
 $Comp
 L Device:LED D2
@@
 F 2 "LED_SMD:LED_0603_1608Metric_Pad1.05x0.95mm_HandSolder" H 9850 2300 60  0001 L CNN
 F 3 "https://datasheet.lcsc.com/szlcsc/Foshan-NationStar-Optoelectronics-FC-DA1608UGK-520D10_C84267.pdf" H 9850 2400 60  0001 L CNN
-F 4 "Optoelectronics" H 9850 2700 60  0001 L CNN "Category"
-F 5 "LED Indication - Discrete" H 9850 2800 60  0001 L CNN "Family"
-F 6 "LED GREEN DIFFUSED" H 9850 3100 60  0001 L CNN "Description"
-F 7 "Active" H 9850 3300 60  0001 L CNN "Status"
-F 8 "C84267" H 9650 2100 50  0001 C CNN "LCSC"
-F 9 "FC-DA1608UGK-520D10" H 9650 2100 50  0001 C CNN "Manufacture PN"
+F 4 "LED GREEN DIFFUSED" H 9850 3100 60  0001 L CNN "Description"
+F 5 "Active" H 9850 3300 60  0001 L CNN "Status"
+F 6 "C84267" H 9650 2100 50  0001 C CNN "LCSC"
 	1    9650 2100
 	-1   0    0    1
 $EndComp
+Wire Wire Line
+	9800 1200 9950 1200
 $EndSCHEMATC
