File: ECAD/PCBs/OH_Specific/Functional/ufc_v4_controller/ufc_v4_controller.sch (KiCad schematic (older format))
At the start: 0 parts

Commit message: Added UFC Controller PCB
Parts:
- added C1: 10uF, Capacitor_SMD:CP_Elec_4x5.3, symbol Device:CP_Small
- added C2: 100nF, Capacitor_SMD:C_0402_1005Metric, symbol Device:C_Small
- added J1: PWR IN, Connector_Molex:Molex_Mini-Fit_Jr_5569-08A2_2x04_P4.20mm_Horizontal, symbol Connector_Generic:Conn_02x04_Top_Bottom
- added J2: MAIN PWR OUT, Connector_Molex:Molex_Mini-Fit_Jr_5566-04A_2x02_P4.20mm_Vertical, symbol Connector_Generic:Conn_02x02_Odd_Even
- added J3: MAIN UFC I/O, Connector_PinHeader_2.54mm:PinHeader_2x07_P2.54mm_Vertical, symbol Connector_Generic:Conn_02x07_Odd_Even
- added J4: UFC PANEL SW, Connector_PinHeader_2.54mm:PinHeader_2x07_P2.54mm_Vertical, symbol Connector_Generic:Conn_02x07_Odd_Even
- added J5: HUD BIT TEST, Connector_PinHeader_2.54mm:PinHeader_1x04_P2.54mm_Horizontal, symbol Connector:Conn_01x04_Male
- added J6: AP PANEL I/O, Connector_PinHeader_2.54mm:PinHeader_2x08_P2.54mm_Vertical, symbol Connector_Generic:Conn_02x08_Odd_Even
- added J7: HUD PANEL I/O, Connector_PinHeader_2.54mm:PinHeader_2x08_P2.54mm_Vertical, symbol Connector_Generic:Conn_02x08_Odd_Even
- added MK1, MK2, MK3, MK4, MK5, MK6: MH, Socket_Arduino_Mega:Arduino_1pin, symbol Mechanical:MountingHole
- added P1: Digital, Connector_PinHeader_2.54mm:PinHeader_2x18_P2.54mm_Vertical, symbol Connector_Generic:Conn_02x18_Odd_Even
- added P2: Power, Connector_PinHeader_2.54mm:PinHeader_1x08_P2.54mm_Vertical, symbol Connector_Generic:Conn_01x08
- added P3, P4: Analog, Connector_PinHeader_2.54mm:PinHeader_1x08_P2.54mm_Vertical, symbol Connector_Generic:Conn_01x08
- added P5: PWM, Connector_PinHeader_2.54mm:PinHeader_1x10_P2.54mm_Vertical, symbol Connector_Generic:Conn_01x10
- added P6: PWM, Connector_PinHeader_2.54mm:PinHeader_1x08_P2.54mm_Vertical, symbol Connector_Generic:Conn_01x08
- added P7: Communication, Connector_PinHeader_2.54mm:PinHeader_1x08_P2.54mm_Vertical, symbol Connector_Generic:Conn_01x08
- added R1: 25.5K, Resistor_SMD:R_0603_1608Metric, symbol Device:R
- added R2: 10K, Resistor_SMD:R_0603_1608Metric, symbol Device:R
- added TP1: TP-12, TestPoint:TestPoint_THTPad_D1.5mm_Drill0.7mm, symbol Connector:TestPoint_Alt
- added TP2: TP-5V, TestPoint:TestPoint_THTPad_D1.5mm_Drill0.7mm, symbol Connector:TestPoint_Alt
- added TP4: TP-GND, TestPoint:TestPoint_THTPad_D1.5mm_Drill0.7mm, symbol Connector:TestPoint_Alt
- added U1: MAX7219EWG+T, Package_SO:SOIC-24W_7.5x15.4mm_P1.27mm, symbol KiCadCustomLib:MAX7219EWG+T
Connections:
- new net: R1.2, U1.18 (ISET)
- new net +12V_SUPPLY: J1.3 (Pin_3), J1.4 (Pin_4), J1.8 (Pin_8), P2.8 (Pin_8), TP1.1
- new net +3V3: P2.4 (Pin_4)
- new net +5V: J4.13 (Pin_13), J7.14 (Pin_14), P2.5 (Pin_5)
- new net +5VD: P1.35 (Pin_35), P1.36 (Pin_36)
- new net +5V_SUPPLY: C1.1, C2.1, J1.6 (Pin_6), J1.7 (Pin_7), J2.1 (Pin_1), J2.2 (Pin_2), R1.1, TP2.1, U1.19 (V+)
- new net 0(Rx0): P6.8 (Pin_8)
- new net 1(Tx0): P6.7 (Pin_7)
- new net 10(**): P5.8 (Pin_8)
- new net 11(**): P5.7 (Pin_7)
- new net 12(**): P5.6 (Pin_6)
- new net 13(**): P5.5 (Pin_5)
- new net 14(Tx3): P7.1 (Pin_1)
- new net 15(Rx3): P7.2 (Pin_2)
- new net 16(Tx2): P7.3 (Pin_3)
- new net 17(Rx2): P7.4 (Pin_4)
- new net 18(Tx1): P7.5 (Pin_5)
- new net 19(Rx1): P7.6 (Pin_6)
- new net 2(**): J5.3 (Pin_3), P6.6 (Pin_6)
- new net 20(SDA): P7.7 (Pin_7)
- new net 21(SCL): P7.8 (Pin_8)
- new net 22: J6.13 (Pin_13), P1.33 (Pin_33)
- new net 23: J6.9 (Pin_9), P1.34 (Pin_34)
- new net 24: J6.11 (Pin_11), P1.31 (Pin_31)
- new net 25: J6.7 (Pin_7), P1.32 (Pin_32)
- new net 26: J7.12 (Pin_12), P1.29 (Pin_29)
- new net 27: J6.5 (Pin_5), P1.30 (Pin_30)
- new net 28: J7.10 (Pin_10), P1.27 (Pin_27)
- new net 29: J6.3 (Pin_3), P1.28 (Pin_28)
- new net 3(**): J5.2 (Pin_2), P6.5 (Pin_5)
- new net 30: J7.8 (Pin_8), P1.25 (Pin_25)
- new net 31: J6.1 (Pin_1), P1.26 (Pin_26)
- new net 32: J7.6 (Pin_6), P1.23 (Pin_23)
- new net 33: J7.15 (Pin_15), P1.24 (Pin_24)
- new net 34: J7.4 (Pin_4), P1.21 (Pin_21)
- new net 35: J7.13 (Pin_13), P1.22 (Pin_22)
- new net 36: J7.2 (Pin_2), P1.19 (Pin_19)
- new net 37: J7.11 (Pin_11), P1.20 (Pin_20)
- new net 38: J3.14 (Pin_14), P1.17 (Pin_17)
- new net 39: J7.9 (Pin_9), P1.18 (Pin_18)
- new net 4(**): J5.1 (Pin_1), P6.4 (Pin_4)
- new net 40: J3.12 (Pin_12), P1.15 (Pin_15)
- new net 41: J3.13 (Pin_13), P1.16 (Pin_16)
- new net 42: J3.10 (Pin_10), P1.13 (Pin_13)
- new net 43: J3.11 (Pin_11), P1.14 (Pin_14)
- new net 44: J3.8 (Pin_8), P1.11 (Pin_11)
- new net 45: J3.9 (Pin_9), P1.12 (Pin_12)
- new net 46: J3.6 (Pin_6), P1.9 (Pin_9)
- new net 47: J3.7 (Pin_7), P1.10 (Pin_10)
- new net 48: J3.4 (Pin_4), P1.7 (Pin_7)
- new net 49: J3.5 (Pin_5), P1.8 (Pin_8)
- new net 5(**): P6.3 (Pin_3)
- new net 50(MISO): P1.5 (Pin_5)
- new net 51(MOSI): P1.6 (Pin_6), U1.1 (DIN)
- new net 52(SCK): J3.2 (Pin_2), P1.3 (Pin_3), U1.13 (CLK)
- new net 53(SS): J3.1 (Pin_1), P1.4 (Pin_4), R2.1, U1.12 (LOAD(~CS))
- new net 6(**): P6.2 (Pin_2)
- new net 7(**): P6.1 (Pin_1)
- new net 8(**): P5.10 (Pin_10)
- new net 9(**): P5.9 (Pin_9)
- new net A0: J7.1 (Pin_1), P3.1 (Pin_1)
- new net A1: J7.3 (Pin_3), P3.2 (Pin_2)
- new net A10: J4.3 (Pin_3), P4.3 (Pin_3)
- new net A11: J4.5 (Pin_5), P4.4 (Pin_4)
- new net A12: J4.7 (Pin_7), P4.5 (Pin_5)
- new net A13: J4.9 (Pin_9), P4.6 (Pin_6)
- new net A14: J4.11 (Pin_11), P4.7 (Pin_7)
- new net A15: P4.8 (Pin_8)
- new net A2: J7.5 (Pin_5), P3.3 (Pin_3)
- new net A3: J7.7 (Pin_7), P3.4 (Pin_4)
- new net A4: J4.2 (Pin_2), P3.5 (Pin_5)
- new net A5: J4.4 (Pin_4), P3.6 (Pin_6)
- new net A6: J4.6 (Pin_6), P3.7 (Pin_7)
- new net A7: J4.8 (Pin_8), P3.8 (Pin_8)
- new net A8: J4.10 (Pin_10), P4.1 (Pin_1)
- new net A9: J4.1 (Pin_1), P4.2 (Pin_2)
- new net AREF: P5.3 (Pin_3)
- new net DIG0: J6.2 (Pin_2), U1.2 (DIG0)
- new net DIG1: U1.11 (DIG1)
- new net DIG2: U1.6 (DIG2)
- new net DIG3: U1.7 (DIG3)
- new net DIG4: U1.3 (DIG4)
- new net DIG5: U1.10 (DIG5)
- new net DIG6: U1.5 (DIG6)
- new net DIG7: U1.8 (DIG7)
- new net DIN2: J3.3 (Pin_3), U1.24 (DOUT)
- new net GND: C1.2, C2.2, J1.1 (Pin_1), J1.2 (Pin_2), J2.3 (Pin_3), J2.4 (Pin_4), J4.12 (Pin_12), J4.14 (Pin_14), J5.4 (Pin_4), J6.15 (Pin_15), J7.16 (Pin_16), P1.1 (Pin_1), P1.2 (Pin_2), P2.6 (Pin_6), P2.7 (Pin_7), P5.4 (Pin_4), R2.2, TP4.1, U1.4 (GND), U1.9 (GND)
- new net IOREF: P2.2 (Pin_2)
- new net Reset: P2.3 (Pin_3)
- new net SCL: P5.1 (Pin_1)
- new net SDA: P5.2 (Pin_2)
- new net SEGA: J6.6 (Pin_6), U1.14 (SegA)
- new net SEGB: J6.8 (Pin_8), U1.16 (SegB)
- new net SEGC: J6.10 (Pin_10), U1.20 (SegC)
- new net SEGD: J6.12 (Pin_12), U1.23 (SegD)
- new net SEGDP: J6.4 (Pin_4), U1.22 (SegDP)
- new net SEGE: J6.14 (Pin_14), U1.21 (SegE)
- new net SEGF: J6.16 (Pin_16), U1.15 (SegF)
- new net SEGG: U1.17 (SegG)
- no-connect marks 0 -> 36
Other:
- note added: "1"
- note added: "1) XXXX"
- note added: "A"
- note added: "A/P BL"
- note added: "A/P SW"
- note added: "ADF 1 (UP)"
- note added: "ADF 2 (DN)"
- note added: "ALT 1 (UP)"
- note added: "ALT 2 (DN)"
- note added: "AOA POT"
- note added: "AP PANEL BL"
- note added: "ARDUINO MEGA REV3"
- note added: "ATT 1 (UP)"
- note added: "ATT 2 (DN)"
- note added: "B"
- note added: "BAL POT"
- note added: "BCN BL"
- note added: "BCN SW"
- note added: "BIT TEST SW"
- note added: "BL COM"
- note added: "BLK LVL POT"
- note added: "BRT POT"
- note added: "CLK & SCK\nMUST BE\nCONNECTED\nIN PARALLEL"
- note added: "COMM1\nENC"
- note added: "COMM2\nENC"
- note added: "D/L BL"
- note added: "D/L SW"
- note added: "DAY/NGT 1 (UP)"
- note added: "DAY/NGT 2 (DN)"
- note added: "EMCON SW"
- note added: "GND"
- note added: "GO LED"
- note added: "I/P SW"
- note added: "IFF BL"
- note added: "IFF SW"
- note added: "ILS BL"
- note added: "ILS SW"
- note added: "KEY MTX COL 1"
- note added: "KEY MTX COL 2"
- note added: "KEY MTX COL 3"
- note added: "KEY MTX COL 4"
- note added: "KEY MTX ROW 1"
- note added: "KEY MTX ROW 2"
- note added: "KEY MTX ROW 3"
- note added: "KEY MTX ROW 4"
- note added: "KEY MTX ROW 5"
- note added: "MOUNT HOLES"
- note added: "NC"
- note added: "NO-GO LED"
- note added: "NORM 1 (UP)"
- note added: "NORM 2 (DN)"
- note added: "NOTE: +5VD NET IS SAME \nAS +5V NET. IT IS BROKEN \nOUT TO SIMPLIFY ROUTING."
- note added: "NOTES: (UNLESS OTHERWISE SPECIFIED)"
- note added: "ON/OFF BL"
- note added: "ON/OFF SW"
- note added: "POWER/BL IN"
- note added: "PWR FLAGS"
- note added: "SW"
- note added: "SW COM"
- note added: "TCN BL"
- note added: "TCN SW"
- note added: "TEST POINTS"
- note added: "VOL1 POT"
- note added: "VOL2 POT"
- note added: "WT BAL 1 (UP)"
- note added: "WT BAL 2 (DN)"
