File: ECAD/PCBs/OH_Specific/Backlighting/RWR_Panel_PCB_V1/RWR_Control_Panel.sch (KiCad schematic (older format))
At the start: 42 parts, among them J1 Conn_01x02, J2 PT_Conn_01x06, J3 Conn_01x02, J4 Conn_01x03, J5 Conn_01x04, J6 Conn_01x03, J7 PT_Conn_01x06, J8 Conn_01x04_Female, J9 Conn_01x04_Female, SW1 PT_Tactile_Switch_Led, SW2 PT_Tactile_Switch_Led, SW3 PT_Tactile_Switch_Led, SW4 PT_Tactile_Switch_Led, SW5 PT_Tactile_Switch_Led

Commit message: Latest backlighting changes
Update to multiple PCBs, mainly changing from micro-fit to mini-fit connectors.
Also changing from individual power rails to filled copper planes where possible.
Parts:
- removed D10, D11, D12, D13, D14, D15, D16, D17, D18, D19, D20, D21, D22, D23, D24, D25, D6, D7, D8, D9: WS2812B, WS2812B:LED3535, symbol LED:WS2812B
- removed J1, J3: Conn_01x02, PT_Library_v001:Molex_1x02_P2.54mm_Vertical, symbol Connector_Generic:Conn_01x02
- removed J2: PT_Conn_01x06, PT_Library_v001:Molex_1x06_P2.54mm_Vertical, symbol PT_Symbol_Library_v001:PT_Conn_01x06
- removed J8, J9: Conn_01x04_Female, footprints:Molex_MicroFit_2X2, symbol Connector:Conn_01x04_Female
- removed R1: 150, Resistor_SMD:R_0201_0603Metric, symbol Device:R
- removed R2: 330, Resistor_SMD:R_0201_0603Metric, symbol Device:R
- added D1: FAIl, LED_THT:LED_D3.0mm, symbol Device:LED
- added D3: OFFSET, LED_THT:LED_D3.0mm, symbol Device:LED
- added D5: SPECIAL, LED_THT:LED_D3.0mm, symbol Device:LED
- added D7: DISPLAY, LED_THT:LED_D3.0mm, symbol Device:LED
- added D9: POWER, LED_THT:LED_D3.0mm, symbol Device:LED
- added J1: LED_COL_ROW, Connector_Molex:Molex_KK-254_AE-6410-08A_1x08_P2.54mm_Vertical, symbol Connector:Conn_01x08_Female
- added J6: SWITCH_COL_ROW, Connector_Molex:Molex_KK-254_AE-6410-08A_1x08_P2.54mm_Vertical, symbol Connector:Conn_01x08_Female
- BIT1: renamed from SW1; symbol PT_Symbol_Library_v001:PT_Tactile_Switch_Led -> RWR_Control_Panel-rescue:PT_Tactile_Switch_Led-PT_Symbol_Library_v001
- D10: renamed from D5; footprint Diode_SMD:D_SOD-123 -> Diode_THT:D_A-405_P7.62mm_Horizontal
- D11: renamed from D26; footprint Diode_SMD:D_SOD-123 -> Diode_THT:D_A-405_P7.62mm_Horizontal
- D2: renamed from D1; footprint Diode_SMD:D_SOD-123 -> Diode_THT:D_A-405_P7.62mm_Horizontal
- D4: renamed from D2; footprint Diode_SMD:D_SOD-123 -> Diode_THT:D_A-405_P7.62mm_Horizontal
- D6: renamed from D3; footprint Diode_SMD:D_SOD-123 -> Diode_THT:D_A-405_P7.62mm_Horizontal
- D8: renamed from D4; footprint Diode_SMD:D_SOD-123 -> Diode_THT:D_A-405_P7.62mm_Horizontal
- ENABLE/OFFSET1: renamed from SW2; symbol PT_Symbol_Library_v001:PT_Tactile_Switch_Led -> RWR_Control_Panel-rescue:PT_Tactile_Switch_Led-PT_Symbol_Library_v001
- ENABLE/SPECIAL1: renamed from SW3; symbol PT_Symbol_Library_v001:PT_Tactile_Switch_Led -> RWR_Control_Panel-rescue:PT_Tactile_Switch_Led-PT_Symbol_Library_v001
- J2: renamed from J4; value Conn_01x03 -> DIMMER; footprint PT_Library_v001:Molex_1x03_P2.54mm_Vertical -> Connector_Molex:Molex_KK-254_AE-6410-03A_1x03_P2.54mm_Vertical
- J3: renamed from J6; value Conn_01x03 -> AUDIO; footprint PT_Library_v001:Molex_1x03_P2.54mm_Vertical -> Connector_Molex:Molex_KK-254_AE-6410-03A_1x03_P2.54mm_Vertical
- J4: renamed from J7; value PT_Conn_01x06 -> ROTARY_SWITCH; footprint PT_Library_v001:Molex_1x06_P2.54mm_Vertical -> Connector_Molex:Molex_KK-254_AE-6410-06A_1x06_P2.54mm_Vertical; symbol PT_Symbol_Library_v001:PT_Conn_01x06 -> RWR_Control_Panel-rescue:PT_Conn_01x06-PT_Symbol_Library_v001
- J5: value Conn_01x04 -> ANALOG; footprint PT_Library_v001:Molex_1x04_P2.54mm_Vertical -> Connector_Molex:Molex_KK-254_AE-6410-04A_1x04_P2.54mm_Vertical
- LIMIT/DISPLAY1: renamed from SW4; symbol PT_Symbol_Library_v001:PT_Tactile_Switch_Led -> RWR_Control_Panel-rescue:PT_Tactile_Switch_Led-PT_Symbol_Library_v001
- POWER1: renamed from SW5; symbol PT_Symbol_Library_v001:PT_Tactile_Switch_Led -> RWR_Control_Panel-rescue:PT_Tactile_Switch_Led-PT_Symbol_Library_v001
Connections:
- net Col1: now also J6.1 (Pin_1)
- net Col2: now also J6.2 (Pin_2)
- net Row1: now also J6.3 (Pin_3)
- net Row2: now also J6.4 (Pin_4)
- net Row3: now also J6.5 (Pin_5)
- net Row4: now also J6.6 (Pin_6)
- net Row5: now also J6.7 (Pin_7)
- net ledcol1: now reaches BIT1.5 (+)
- net ledcol1: now also ENABLE/OFFSET1.5 (+), ENABLE/SPECIAL1.5 (+), LIMIT/DISPLAY1.5 (+), POWER1.5 (+), J1.1 (Pin_1)
- net ledrow1: now reaches BIT1.6 (-)
- net ledrow1: now also D1.1 (K), J1.3 (Pin_3); no longer ENABLE/OFFSET1.5 (+)
- net ledrow2: now reaches ENABLE/OFFSET1.6 (-)
- net ledrow2: now also D3.1 (K), J1.4 (Pin_4); no longer ENABLE/SPECIAL1.5 (+)
- net ledrow4: now reaches LIMIT/DISPLAY1.6 (-)
- net ledrow4: now also D7.1 (K), J1.6 (Pin_6); no longer POWER1.5 (+)
- net BckltGND renamed ledrow3
- net ledrow3: now also D5.1 (K), J1.5 (Pin_5); no longer POWER1.6 (-)
- new net ledcol2: D1.2 (A), D3.2 (A), D5.2 (A), D7.2 (A), D9.2 (A), J1.2 (Pin_2)
- new net ledrow5: D9.1 (K), J1.7 (Pin_7), POWER1.6 (-)
- no-connect marks 0 -> 2
Other:
- note removed: "Backlighting"
