File: ECAD/PCBs/OH_Specific/Backlighting/SPIN_RCV_Panel_PCB_V1/SPIN RCV Panel PCB V1.sch (KiCad schematic (older format))
At the start: 86 parts, among them J1 Conn_01x04_Female, J2 Conn_01x04_Female

Commit message: Latest backlighting changes
Update to multiple PCBs, mainly changing from micro-fit to mini-fit connectors.
Also changing from individual power rails to filled copper planes where possible.
Parts:
- D25, D29, D30, D32, D33, D34, D35, D36, D37, D39, D40, D44, D45, D49, D51, D53: footprint OH_Backlighting:LED_WS2812B_MINI_PLCC4_3.5x3.5mm_P1.75mm -> LED_SMD:LED_SK6812MINI_PLCC4_3.5x3.5mm_P1.75mm
Changed lines of the file:
@@
 F 0 "D25" H 10344 2991 50  0000 L CNN
 F 1 "WS2812B" H 10344 2900 50  0000 L CNN
-F 2 "OH_Backlighting:LED_WS2812B_MINI_PLCC4_3.5x3.5mm_P1.75mm" H 10050 2600 50  0001 L TNN
+F 2 "LED_SMD:LED_SK6812MINI_PLCC4_3.5x3.5mm_P1.75mm" H 10050 2600 50  0001 L TNN
 F 3 "https://cdn-shop.adafruit.com/datasheets/WS2812B.pdf" H 10100 2525 50  0001 L TNN
 F 4 "C114586" H 10344 2809 50  0000 L CNN "LCSC Part Number"
@@
 F 0 "D29" H 4144 3891 50  0000 L CNN
 F 1 "WS2812B" H 4144 3800 50  0000 L CNN
-F 2 "OH_Backlighting:LED_WS2812B_MINI_PLCC4_3.5x3.5mm_P1.75mm" H 3850 3500 50  0001 L TNN
+F 2 "LED_SMD:LED_SK6812MINI_PLCC4_3.5x3.5mm_P1.75mm" H 3850 3500 50  0001 L TNN
 F 3 "https://cdn-shop.adafruit.com/datasheets/WS2812B.pdf" H 3900 3425 50  0001 L TNN
 F 4 "C114586" H 4144 3709 50  0000 L CNN "LCSC Part Number"
@@
 F 0 "D30" H 4894 3891 50  0000 L CNN
 F 1 "WS2812B" H 4894 3800 50  0000 L CNN
-F 2 "OH_Backlighting:LED_WS2812B_MINI_PLCC4_3.5x3.5mm_P1.75mm" H 4600 3500 50  0001 L TNN
+F 2 "LED_SMD:LED_SK6812MINI_PLCC4_3.5x3.5mm_P1.75mm" H 4600 3500 50  0001 L TNN
 F 3 "https://cdn-shop.adafruit.com/datasheets/WS2812B.pdf" H 4650 3425 50  0001 L TNN
 F 4 "C114586" H 4894 3709 50  0000 L CNN "LCSC Part Number"
@@
 F 0 "D32" H 6494 3891 50  0000 L CNN
 F 1 "WS2812B" H 6494 3800 50  0000 L CNN
-F 2 "OH_Backlighting:LED_WS2812B_MINI_PLCC4_3.5x3.5mm_P1.75mm" H 6200 3500 50  0001 L TNN
+F 2 "LED_SMD:LED_SK6812MINI_PLCC4_3.5x3.5mm_P1.75mm" H 6200 3500 50  0001 L TNN
 F 3 "https://cdn-shop.adafruit.com/datasheets/WS2812B.pdf" H 6250 3425 50  0001 L TNN
 F 4 "C114586" H 6494 3709 50  0000 L CNN "LCSC Part Number"
@@
 F 0 "D33" H 7244 3891 50  0000 L CNN
 F 1 "WS2812B" H 7244 3800 50  0000 L CNN
-F 2 "OH_Backlighting:LED_WS2812B_MINI_PLCC4_3.5x3.5mm_P1.75mm" H 6950 3500 50  0001 L TNN
+F 2 "LED_SMD:LED_SK6812MINI_PLCC4_3.5x3.5mm_P1.75mm" H 6950 3500 50  0001 L TNN
 F 3 "https://cdn-shop.adafruit.com/datasheets/WS2812B.pdf" H 7000 3425 50  0001 L TNN
 F 4 "C114586" H 7244 3709 50  0000 L CNN "LCSC Part Number"
@@
 F 0 "D34" H 8044 3891 50  0000 L CNN
 F 1 "WS2812B" H 8044 3800 50  0000 L CNN
-F 2 "OH_Backlighting:LED_WS2812B_MINI_PLCC4_3.5x3.5mm_P1.75mm" H 7750 3500 50  0001 L TNN
+F 2 "LED_SMD:LED_SK6812MINI_PLCC4_3.5x3.5mm_P1.75mm" H 7750 3500 50  0001 L TNN
 F 3 "https://cdn-shop.adafruit.com/datasheets/WS2812B.pdf" H 7800 3425 50  0001 L TNN
 F 4 "C114586" H 8044 3709 50  0000 L CNN "LCSC Part Number"
@@
 F 0 "D36" H 9544 3891 50  0000 L CNN
 F 1 "WS2812B" H 9544 3800 50  0000 L CNN
-F 2 "OH_Backlighting:LED_WS2812B_MINI_PLCC4_3.5x3.5mm_P1.75mm" H 9250 3500 50  0001 L TNN
+F 2 "LED_SMD:LED_SK6812MINI_PLCC4_3.5x3.5mm_P1.75mm" H 9250 3500 50  0001 L TNN
 F 3 "https://cdn-shop.adafruit.com/datasheets/WS2812B.pdf" H 9300 3425 50  0001 L TNN
 F 4 "C114586" H 9544 3709 50  0000 L CNN "LCSC Part Number"
@@
 F 0 "D37" H 10344 3891 50  0000 L CNN
 F 1 "WS2812B" H 10344 3800 50  0000 L CNN
-F 2 "OH_Backlighting:LED_WS2812B_MINI_PLCC4_3.5x3.5mm_P1.75mm" H 10050 3500 50  0001 L TNN
+F 2 "LED_SMD:LED_SK6812MINI_PLCC4_3.5x3.5mm_P1.75mm" H 10050 3500 50  0001 L TNN
 F 3 "https://cdn-shop.adafruit.com/datasheets/WS2812B.pdf" H 10100 3425 50  0001 L TNN
 F 4 "C114586" H 10344 3709 50  0000 L CNN "LCSC Part Number"
@@
 F 0 "D35" H 8794 3891 50  0000 L CNN
 F 1 "WS2812B" H 8794 3800 50  0000 L CNN
-F 2 "OH_Backlighting:LED_WS2812B_MINI_PLCC4_3.5x3.5mm_P1.75mm" H 8500 3500 50  0001 L TNN
+F 2 "LED_SMD:LED_SK6812MINI_PLCC4_3.5x3.5mm_P1.75mm" H 8500 3500 50  0001 L TNN
 F 3 "https://cdn-shop.adafruit.com/datasheets/WS2812B.pdf" H 8550 3425 50  0001 L TNN
 F 4 "C114586" H 8794 3709 50  0000 L CNN "LCSC Part Number"
@@
 F 0 "D39" H 2644 4841 50  0000 L CNN
 F 1 "WS2812B" H 2644 4750 50  0000 L CNN
-F 2 "OH_Backlighting:LED_WS2812B_MINI_PLCC4_3.5x3.5mm_P1.75mm" H 2350 4450 50  0001 L TNN
+F 2 "LED_SMD:LED_SK6812MINI_PLCC4_3.5x3.5mm_P1.75mm" H 2350 4450 50  0001 L TNN
 F 3 "https://cdn-shop.adafruit.com/datasheets/WS2812B.pdf" H 2400 4375 50  0001 L TNN
 F 4 "C114586" H 2644 4659 50  0000 L CNN "LCSC Part Number"
@@
 F 0 "D40" H 3444 4841 50  0000 L CNN
 F 1 "WS2812B" H 3444 4750 50  0000 L CNN
-F 2 "OH_Backlighting:LED_WS2812B_MINI_PLCC4_3.5x3.5mm_P1.75mm" H 3150 4450 50  0001 L TNN
+F 2 "LED_SMD:LED_SK6812MINI_PLCC4_3.5x3.5mm_P1.75mm" H 3150 4450 50  0001 L TNN
 F 3 "https://cdn-shop.adafruit.com/datasheets/WS2812B.pdf" H 3200 4375 50  0001 L TNN
 F 4 "C114586" H 3444 4659 50  0000 L CNN "LCSC Part Number"
@@
 F 0 "D44" H 6544 4841 50  0000 L CNN
 F 1 "WS2812B" H 6544 4750 50  0000 L CNN
-F 2 "OH_Backlighting:LED_WS2812B_MINI_PLCC4_3.5x3.5mm_P1.75mm" H 6250 4450 50  0001 L TNN
+F 2 "LED_SMD:LED_SK6812MINI_PLCC4_3.5x3.5mm_P1.75mm" H 6250 4450 50  0001 L TNN
 F 3 "https://cdn-shop.adafruit.com/datasheets/WS2812B.pdf" H 6300 4375 50  0001 L TNN
 F 4 "C114586" H 6544 4659 50  0000 L CNN "LCSC Part Number"
@@
 F 0 "D45" H 7294 4841 50  0000 L CNN
 F 1 "WS2812B" H 7294 4750 50  0000 L CNN
-F 2 "OH_Backlighting:LED_WS2812B_MINI_PLCC4_3.5x3.5mm_P1.75mm" H 7000 4450 50  0001 L TNN
+F 2 "LED_SMD:LED_SK6812MINI_PLCC4_3.5x3.5mm_P1.75mm" H 7000 4450 50  0001 L TNN
 F 3 "https://cdn-shop.adafruit.com/datasheets/WS2812B.pdf" H 7050 4375 50  0001 L TNN
 F 4 "C114586" H 7294 4659 50  0000 L CNN "LCSC Part Number"
@@
 F 0 "D51" H 2594 5741 50  0000 L CNN
 F 1 "WS2812B" H 2594 5650 50  0000 L CNN
-F 2 "OH_Backlighting:LED_WS2812B_MINI_PLCC4_3.5x3.5mm_P1.75mm" H 2300 5350 50  0001 L TNN
+F 2 "LED_SMD:LED_SK6812MINI_PLCC4_3.5x3.5mm_P1.75mm" H 2300 5350 50  0001 L TNN
 F 3 "https://cdn-shop.adafruit.com/datasheets/WS2812B.pdf" H 2350 5275 50  0001 L TNN
 F 4 "C114586" H 2594 5559 50  0000 L CNN "LCSC Part Number"
@@
 F 0 "D53" H 4144 5741 50  0000 L CNN
 F 1 "WS2812B" H 4144 5650 50  0000 L CNN
-F 2 "OH_Backlighting:LED_WS2812B_MINI_PLCC4_3.5x3.5mm_P1.75mm" H 3850 5350 50  0001 L TNN
+F 2 "LED_SMD:LED_SK6812MINI_PLCC4_3.5x3.5mm_P1.75mm" H 3850 5350 50  0001 L TNN
 F 3 "https://cdn-shop.adafruit.com/datasheets/WS2812B.pdf" H 3900 5275 50  0001 L TNN
 F 4 "C114586" H 4144 5559 50  0000 L CNN "LCSC Part Number"
@@
 F 0 "D49" H 10394 4841 50  0000 L CNN
 F 1 "WS2812B" H 10394 4750 50  0000 L CNN
-F 2 "OH_Backlighting:LED_WS2812B_MINI_PLCC4_3.5x3.5mm_P1.75mm" H 10100 4450 50  0001 L TNN
+F 2 "LED_SMD:LED_SK6812MINI_PLCC4_3.5x3.5mm_P1.75mm" H 10100 4450 50  0001 L TNN
 F 3 "https://cdn-shop.adafruit.com/datasheets/WS2812B.pdf" H 10150 4375 50  0001 L TNN
 F 4 "C114586" H 10394 4659 50  0000 L CNN "LCSC Part Number"
