File: ECAD/PCBs/OH_Specific/Functional/ampcd_button_board/_autosave-ampcd_button_board.sch (KiCad schematic (older format))
At the start: 79 parts, among them J1 Conn_01x06, SW1 TL1240GQ, SW10 TL1240GQ, SW11 TL1240GQ, SW12 TL1240GQ, SW13 TL1240GQ, SW14 TL1240GQ, SW15 TL1240GQ, SW16 TL1240GQ, SW17 TL1240GQ, SW18 TL1240GQ, SW19 TL1240GQ, SW2 TL1240GQ, SW20 TL1240GQ, SW21 TL1240GQ, SW22 TL1240GQ, SW23 TL1240GQ, SW24 TL1240GQ, SW25 TL1240GQ, SW26 TL1240GQ, SW27 TL1240GQ, SW28 TL1240GQ, SW3 TL1240GQ, SW4 TL1240GQ, SW5 TL1240GQ, SW6 TL1240GQ, SW7 TL1240GQ, SW8 TL1240GQ, SW9 TL1240GQ, U1 TCA9554PWR, U2 TCA9554PWR, U3 TCA9554PWR, U4 TCA9554PWR

Commit message: Preliminary AMPCD Component layout
Starting work on the AMPCD PCB layout in earnest.
Parts:
- J1: footprint Connector_Molex:Molex_KK-254_AE-6410-06A_1x06_P2.54mm_Vertical -> Connector_PinHeader_2.54mm:PinHeader_1x06_P2.54mm_Horizontal; PN 22292061 -> (none)
Changed lines of the file:
@@
 F 0 "J1" H 5900 1800 50  0000 C CNN
 F 1 "Conn_01x06" H 5900 1700 50  0000 C CNN
-F 2 "Connector_Molex:Molex_KK-254_AE-6410-06A_1x06_P2.54mm_Vertical" H 5900 1350 50  0001 C CNN
-F 3 "https://www.molex.com/pdm_docs/sd/022292061_sd.pdf" H 5900 1350 50  0001 C CNN
-F 4 "22292061" H 5900 1350 50  0001 C CNN "PN"
+F 2 "Connector_PinHeader_2.54mm:PinHeader_1x06_P2.54mm_Horizontal" H 5900 1350 50  0001 C CNN
+F 3 "" H 5900 1350 50  0001 C CNN
+F 4 "" H 5900 1350 50  0001 C CNN "PN"
 	1    5900 1350
 	1    0    0    -1
