File: ECAD/PCBs/OH_Specific/Backlighting/Landing_Gear_Panel_PCB_V2/Landing Gear Panel PCB V2.sch (KiCad schematic (older format))
At the start: 49 parts, among them J1 Conn_01x04_Female, J2 Conn_01x04_Female

Commit message: Landing Gear Panel Backlighting Update
Added - Assembly note silkscreen about connector soldering
Added - H6 + H7 hole silkscreen labels.
Changed - Board outline to match the backplate, resulting in it sitting on top of the AUX panel.
Changed - Version from 2.1 to 2.2
Changed - Manufacturing files to match changes.
Removed - Little power cleaning capacitor 22, the cutout in the backplate was too large to be covered by the lightplate, resulting in it being visible when viewed from the front.
Parts:
- removed C22: C, Capacitor_SMD:C_0603_1608Metric, symbol Device:C
- C1: symbol Device:C_Polarized -> Landing-Gear-Panel-PCB-V2-rescue:C_Polarized-Device
- C10, C11, C12, C13, C14, C15, C16, C17, C18, C19, C2, C20, C21, C3, C4, C5, C6, C7, C8, C9: symbol Device:C -> Landing-Gear-Panel-PCB-V2-rescue:C-Device
- D1, D10, D11, D12, D13, D14, D15, D16, D17, D18, D19, D2, D20, D21, D22, D23, D3, D4, D5, D6, D7, D8, D9: symbol LED:WS2812B -> Landing-Gear-Panel-PCB-V2-rescue:WS2812B-LED
- D24: symbol Device:LED -> Landing-Gear-Panel-PCB-V2-rescue:LED-Device
- J1, J2: symbol Connector:Conn_01x04_Female -> Landing-Gear-Panel-PCB-V2-rescue:Conn_01x04_Female-Connector
- R1: symbol Device:R -> Landing-Gear-Panel-PCB-V2-rescue:R-Device
Connections:
- wire segments 156 -> 154
Changed lines of the file:
@@
 $EndDescr
 $Comp
-L Connector:Conn_01x04_Female J2
+L Landing-Gear-Panel-PCB-V2-rescue:Conn_01x04_Female-Connector J2
 U 1 1 5F87F05B
 P 5050 550
@@
 $EndComp
 $Comp
-L Connector:Conn_01x04_Female J1
+L Landing-Gear-Panel-PCB-V2-rescue:Conn_01x04_Female-Connector J1
 U 1 1 5F880577
 P 5550 550
@@
 $EndComp
 $Comp
-L LED:WS2812B D1
+L Landing-Gear-Panel-PCB-V2-rescue:WS2812B-LED D1
 U 1 1 5F88255D
 P 5200 1550
@@
 $EndComp
 $Comp
-L LED:WS2812B D2
+L Landing-Gear-Panel-PCB-V2-rescue:WS2812B-LED D2
 U 1 1 5F883FB6
 P 6150 1550
@@
 $EndComp
 $Comp
-L LED:WS2812B D3
+L Landing-Gear-Panel-PCB-V2-rescue:WS2812B-LED D3
 U 1 1 5F885B92
 P 7150 1550
@@
 $EndComp
 $Comp
-L LED:WS2812B D4
+L Landing-Gear-Panel-PCB-V2-rescue:WS2812B-LED D4
 U 1 1 5F887524
 P 4150 2450
@@
 $EndComp
 $Comp
-L LED:WS2812B D5
+L Landing-Gear-Panel-PCB-V2-rescue:WS2812B-LED D5
 U 1 1 5F88796A
 P 5050 2450
@@
 $EndComp
 $Comp
-L LED:WS2812B D6
+L Landing-Gear-Panel-PCB-V2-rescue:WS2812B-LED D6
 U 1 1 5F8894DE
 P 6150 2450
@@
 $EndComp
 $Comp
-L LED:WS2812B D7
+L Landing-Gear-Panel-PCB-V2-rescue:WS2812B-LED D7
 U 1 1 5F889812
 P 7150 2450
@@
 $EndComp
 $Comp
-L LED:WS2812B D8
+L Landing-Gear-Panel-PCB-V2-rescue:WS2812B-LED D8
 U 1 1 5F889E26
 P 8100 2450
@@
 $EndComp
 $Comp
-L LED:WS2812B D9
+L Landing-Gear-Panel-PCB-V2-rescue:WS2812B-LED D9
 U 1 1 5F88A704
 P 5050 3300
@@
 $EndComp
 $Comp
-L LED:WS2812B D10
+L Landing-Gear-Panel-PCB-V2-rescue:WS2812B-LED D10
 U 1 1 5F88ADC8
 P 6150 3300
@@
 $EndComp
 $Comp
-L LED:WS2812B D11
+L Landing-Gear-Panel-PCB-V2-rescue:WS2812B-LED D11
 U 1 1 5F88B38C
 P 7150 3300
@@
 $EndComp
 $Comp
-L LED:WS2812B D12
+L Landing-Gear-Panel-PCB-V2-rescue:WS2812B-LED D12
 U 1 1 5F88B85A
 P 8100 3300
@@
 $EndComp
 $Comp
-L LED:WS2812B D13
+L Landing-Gear-Panel-PCB-V2-rescue:WS2812B-LED D13
 U 1 1 5F88BFB4
 P 6150 4200
@@
 $EndComp
 $Comp
-L LED:WS2812B D14
+L Landing-Gear-Panel-PCB-V2-rescue:WS2812B-LED D14
 U 1 1 5F88C388
 P 7150 4200
@@
 $EndComp
 $Comp
-L LED:WS2812B D15
+L Landing-Gear-Panel-PCB-V2-rescue:WS2812B-LED D15
 U 1 1 5F88CBDE
 P 8100 4200
@@
 $EndComp
 $Comp
-L LED:WS2812B D17
+L Landing-Gear-Panel-PCB-V2-rescue:WS2812B-LED D17
 U 1 1 5F88E31E
 P 5350 5000
@@
 $EndComp
 $Comp
-L LED:WS2812B D16
+L Landing-Gear-Panel-PCB-V2-rescue:WS2812B-LED D16
 U 1 1 5F88F116
 P 3850 4350
@@
 $EndComp
 $Comp
-L LED:WS2812B D18
+L Landing-Gear-Panel-PCB-V2-rescue:WS2812B-LED D18
 U 1 1 5F88F8AE
 P 3850 5200
@@
 $EndComp
 $Comp
-L LED:WS2812B D19
+L Landing-Gear-Panel-PCB-V2-rescue:WS2812B-LED D19
 U 1 1 5F89017C
 P 2800 5950
@@
 $EndComp
 $Comp
-L LED:WS2812B D20
+L Landing-Gear-Panel-PCB-V2-rescue:WS2812B-LED D20
 U 1 1 5F890D28
 P 4750 5950
@@
 $EndComp
 $Comp
-L LED:WS2812B D21
+L Landing-Gear-Panel-PCB-V2-rescue:WS2812B-LED D21
 U 1 1 5F891AF0
 P 3350 6900
@@
 $EndComp
 $Comp
-L LED:WS2812B D22
+L Landing-Gear-Panel-PCB-V2-rescue:WS2812B-LED D22
 U 1 1 5F892414
 P 4400 6900
@@
 $EndComp
 $Comp
-L LED:WS2812B D23
+L Landing-Gear-Panel-PCB-V2-rescue:WS2812B-LED D23
 U 1 1 5F892E06
 P 5400 7450
@@
 LEDGND
 $Comp
-L Device:LED D24
+L Landing-Gear-Panel-PCB-V2-rescue:LED-Device D24
 U 1 1 5F9C449E
 P 2050 850
@@
 $EndComp
 $Comp
-L Device:R R1
+L Landing-Gear-Panel-PCB-V2-rescue:R-Device R1
 U 1 1 5F9C59BE
 P 1650 1000
@@
 LEDGND
 $Comp
-L Device:C C4
+L Landing-Gear-Panel-PCB-V2-rescue:C-Device C4
 U 1 1 5F9D59B5
 P 6950 5300
@@
 $EndComp
 $Comp
-L Device:C C5
+L Landing-Gear-Panel-PCB-V2-rescue:C-Device C5
 U 1 1 5F9E279A
 P 7250 5300
@@
 $EndComp
 $Comp
-L Device:C C6
+L Landing-Gear-Panel-PCB-V2-rescue:C-Device C6
 U 1 1 5F9E8CA0
 P 7550 5300
@@
 $EndComp
 $Comp
-L Device:C C7
+L Landing-Gear-Panel-PCB-V2-rescue:C-Device C7
 U 1 1 5F9EF184
 P 7850 5300
@@
 $EndComp
 $Comp
-L Device:C C8
+L Landing-Gear-Panel-PCB-V2-rescue:C-Device C8
 U 1 1 5F9F56B9
 P 8150 5300
@@
 $EndComp
 $Comp
-L Device:C C9
+L Landing-Gear-Panel-PCB-V2-rescue:C-Device C9
 U 1 1 5F9FBC5E
 P 8450 5300
@@
 $EndComp
 $Comp
-L Device:C C10
+L Landing-Gear-Panel-PCB-V2-rescue:C-Device C10
 U 1 1 5FA02139
 P 8750 5300
@@
 $EndComp
 $Comp
-L Device:C C11
+L Landing-Gear-Panel-PCB-V2-rescue:C-Device C11
 U 1 1 5FA087F2
 P 9050 5300
@@
 $EndComp
 $Comp
-L Device:C C12
+L Landing-Gear-Panel-PCB-V2-rescue:C-Device C12
 U 1 1 5FA0ECEB
 P 9400 5300
@@
 $EndComp
 $Comp
-L Device:C C13
+L Landing-Gear-Panel-PCB-V2-rescue:C-Device C13
 U 1 1 5FA15297
 P 9700 5300
@@
 $EndComp
 $Comp
-L Device:C C14
+L Landing-Gear-Panel-PCB-V2-rescue:C-Device C14
 U 1 1 5FA1B77A
 P 10000 5300
@@
 $EndComp
 $Comp
-L Device:C C15
+L Landing-Gear-Panel-PCB-V2-rescue:C-Device C15
 U 1 1 5FA21C84
 P 10300 5300
@@
 $EndComp
 $Comp
-L Device:C C16
+L Landing-Gear-Panel-PCB-V2-rescue:C-Device C16
 U 1 1 5FA283D6
 P 10600 5300
@@
 $EndComp
 $Comp
-L Device:C C17
+L Landing-Gear-Panel-PCB-V2-rescue:C-Device C17
 U 1 1 5FA2EA00
 P 10900 5300
@@
 $EndComp
 $Comp
-L Device:C C3
+L Landing-Gear-Panel-PCB-V2-rescue:C-Device C3
 U 1 1 5FA35644
 P 6700 5300
@@
 $EndComp
 $Comp
-L Device:C C2
+L Landing-Gear-Panel-PCB-V2-rescue:C-Device C2
 U 1 1 5FA3BB82
 P 6400 5300
@@
 DATAIN
 $Comp
-L Device:C C18
+L Landing-Gear-Panel-PCB-V2-rescue:C-Device C18
 U 1 1 5FEBD809
 P 11200 5300
@@
 $EndComp
 $Comp
-L Device:C C19
+L Landing-Gear-Panel-PCB-V2-rescue:C-Device C19
 U 1 1 5FEBD80F
 P 11500 5300
@@
 $EndComp
 $Comp
-L Device:C C20
+L Landing-Gear-Panel-PCB-V2-rescue:C-Device C20
 U 1 1 5FEBD815
 P 11800 5300
@@
 	11500 5450 11800 5450
 $Comp
-L Device:C C21
+L Landing-Gear-Panel-PCB-V2-rescue:C-Device C21
 U 1 1 5FEF267C
 P 12100 5300
@@
 	1    0    0    -1
 $EndComp
-$Comp
-L Device:C C22
-U 1 1 5FEF2682
-P 12400 5300
-F 0 "C22" H 12515 5346 50  0000 L CNN
-F 1 "C" H 12515 5255 50  0000 L CNN
-F 2 "Capacitor_SMD:C_0603_1608Metric" H 12438 5150 50  0001 C CNN
-F 3 "~" H 12400 5300 50  0001 C CNN
-	1    12400 5300
-	1    0    0    -1
-$EndComp
+Wire Wire Line
+	12100 5150 11800 5150
+Wire Wire Line
+	11800 5450 12100 5450
+$Comp
+L Landing-Gear-Panel-PCB-V2-rescue:C_Polarized-Device C1
+U 1 1 5F88069E
+P 12450 5300
+F 0 "C1" H 12332 5254 50  0000 R CNN
+F 1 "C_Polarized" H 12332 5345 50  0000 R CNN
+F 2 "Capacitor_SMD:CP_Elec_8x10" H 12488 5150 50  0001 C CNN
+F 3 "~" H 12450 5300 50  0001 C CNN
+	1    12450 5300
+	1    0    0    -1
+$EndComp
+Wire Wire Line
+	12450 5150 12100 5150
 Connection ~ 12100 5150
 Wire Wire Line
-	12100 5150 11800 5150
-Wire Wire Line
-	11800 5450 12100 5450
+	12100 5450 12450 5450
 Connection ~ 12100 5450
-Wire Wire Line
-	12100 5450 12400 5450
-Wire Wire Line
-	12400 5150 12100 5150
-$Comp
-L Device:C_Polarized C1
-U 1 1 5F88069E
-P 12700 5300
-F 0 "C1" H 12582 5254 50  0000 R CNN
-F 1 "C_Polarized" H 12582 5345 50  0000 R CNN
-F 2 "Capacitor_SMD:CP_Elec_8x10" H 12738 5150 50  0001 C CNN
-F 3 "~" H 12700 5300 50  0001 C CNN
-	1    12700 5300
-	1    0    0    -1
-$EndComp
-Wire Wire Line
-	12700 5450 12400 5450
-Wire Wire Line
-	12400 5150 12700 5150
-Connection ~ 12400 5150
-Connection ~ 12400 5450
 $EndSCHEMATC
