File: ECAD/PCBs/ABSIS/ABSIS_PMS/ABSIS_PMS.sch (KiCad schematic (older format))
At the start: 15 parts, among them J1 FROM PSU, J2 FROM SIM PWR, J3 EXT ACC OUT, U1 140817140010, U2 140817140010, U3 140817140010, U4 140817140010

Commit message: Finished PMS, LIP Interconnect 95%
Parts:
- J3: footprint Connector_PinHeader_2.54mm:PinHeader_2x04_P2.54mm_Vertical -> Connector_Molex:Molex_Mini-Fit_Jr_5566-08A2_2x04_P4.20mm_Vertical
Connections:
- net EXT_ACC1+: now also J3.2 (Pin_2); no longer J3.1 (Pin_1)
- net EXT_ACC1-: now also J3.1 (Pin_1); no longer J3.2 (Pin_2)
- net EXT_ACC2+: now also J3.4 (Pin_4); no longer J3.3 (Pin_3)
- net EXT_ACC2-: now also J3.3 (Pin_3); no longer J3.4 (Pin_4)
- net EXT_ACC3+: now also J3.6 (Pin_6); no longer J3.5 (Pin_5)
- net EXT_ACC3-: now also J3.5 (Pin_5); no longer J3.6 (Pin_6)
- net EXT_ACC4+: now also J3.8 (Pin_8); no longer J3.7 (Pin_7)
- net EXT_ACC4-: now also J3.7 (Pin_7); no longer J3.8 (Pin_8)
Changed lines of the file:
@@
 F 0 "J3" H 4300 4750 50  0000 C CNN
 F 1 "EXT ACC OUT" H 4300 4650 50  0000 C CNN
-F 2 "Connector_PinHeader_2.54mm:PinHeader_2x04_P2.54mm_Vertical" H 4200 4200 50  0001 C CNN
+F 2 "Connector_Molex:Molex_Mini-Fit_Jr_5566-08A2_2x04_P4.20mm_Vertical" H 4200 4200 50  0001 C CNN
 F 3 "~" H 4200 4200 50  0001 C CNN
 	1    4200 4200
 	1    0    0    -1
 $EndComp
+Text Label 4400 4000 0    50   ~ 0
+EXT_ACC1+
 Text Label 4400 3900 0    50   ~ 0
-EXT_ACC1+
-Text Label 4400 4000 0    50   ~ 0
 EXT_ACC1-
+Text Label 4400 4200 0    50   ~ 0
+EXT_ACC2+
 Text Label 4400 4100 0    50   ~ 0
-EXT_ACC2+
-Text Label 4400 4200 0    50   ~ 0
 EXT_ACC2-
+Text Label 4400 4400 0    50   ~ 0
+EXT_ACC3+
 Text Label 4400 4300 0    50   ~ 0
-EXT_ACC3+
-Text Label 4400 4400 0    50   ~ 0
 EXT_ACC3-
+Text Label 4400 4600 0    50   ~ 0
+EXT_ACC4+
 Text Label 4400 4500 0    50   ~ 0
-EXT_ACC4+
-Text Label 4400 4600 0    50   ~ 0
 EXT_ACC4-
 Text Label 7950 3850 0    50   ~ 0
