File: ECAD/interconnects/OH_Left_Console.sch (KiCad schematic (older format))
At the start: 354 parts

Commit message: DDI Controller Redesigned with Pro Micro
DDI Controller Redesigned with Pro Micro
LIP Interconnects WIP
Parts:
- removed (0AxAxWx): ABSIS-CA-C-XXX, symbol Connector_Generic:Conn_01x01
- removed (0AxAxWx): USB A TO B, symbol Connector_Generic:Conn_01x01
- removed 4A1W1P? (x2), 4A2A1~ (x9), ~ (x35): ~, symbol Connector_Generic:Conn_01x01
- added (0AxAxWx): ABSIS-CA-C-XXX, symbol Connector_Generic:Conn_01x01
- added (0AxAxWx): USB A TO B, symbol Connector_Generic:Conn_01x01
- added 4A1W1P? (x2), 4A2A1~ (x9), ~ (x35): ~, symbol Connector_Generic:Conn_01x01
Connections:
- net LC<>ABSIS_PSU_PWR: now also (0AxAxWx).1 (Pin_1)
- net LC<>UIP_USB_HUB: now also (0AxAxWx).1 (Pin_1)
- net at 4A14A1W2.1 (Pin_1): now also 4A1W1P?.1 (Pin_1)
- net at 4A3A1.USB: now also 4A2A1~.1 (Pin_1)
- net at 4A5A1A2.J1 (BLC_IN): now also ~.1 (Pin_1)
- net at 4A5A1A2.J2 (BLC_OUT): now also ~.1 (Pin_1)
- net at 4A6A1A2.J2 (BLC_OUT): now also 4A2A1~.1 (Pin_1)
- net at A4A9A1A1.COM1 (COMM_SW): now also ~.1 (Pin_1)
- net at 4A14A1W3.1 (Pin_1): now also 4A1W1P?.1 (Pin_1)
- net at 4A6A1.USB: now also 4A2A1~.1 (Pin_1)
- net at 4A1W1.1 (Pin_1): now also ~.1 (Pin_1)
- net at 4A13A1W1.1 (Pin_1): now also ~.1 (Pin_1)
- net at 4A2A1A2.J2 (BLC_OUT): now also ~.1 (Pin_1)
- net at 4A9A1.J8 (EXT_+5V): now also 4A2A1~.1 (Pin_1)
- net at 4A13A1W8.1 (Pin_1): now also ~.1 (Pin_1)
- net at 4A2A1A2.J1 (BLC_IN): now also ~.1 (Pin_1)
- net at 4A3A1A2.J1 (BLC_IN): now also ~.1 (Pin_1)
- net at 4A7A1A2.J2 (BLC_OUT): now also 4A2A1~.1 (Pin_1)
- net at 4A7A1A2.J1 (BLC_IN): now also 4A2A1~.1 (Pin_1)
- net at 4A7A4A2.J2 (BLC_OUT): now also 4A2A1~.1 (Pin_1)
- net at 4A4A1A2.J2 (BLC_OUT): now also ~.1 (Pin_1)
- net at 10A1A1A2.J1 (BLC_IN): now also ~.1 (Pin_1)
- net at 10A1A1A2.J2 (BLC_OUT): now also ~.1 (Pin_1)
- net at 4A4A2A2.J1 (BLC_IN): now also ~.1 (Pin_1)
- net at 4A4A3A2.J1 (BLC_IN): now also ~.1 (Pin_1)
- net at 4A4A3A2.J2 (BLC_OUT): now also ~.1 (Pin_1)
- net at 4A1W12.1 (Pin_1): now also ~.1 (Pin_1)
- net at A4A9A1A1.ANT1 (ANT_ELEV): now also ~.1 (Pin_1)
- net at A4A9A1A1.CM1 (CM_SW): now also ~.1 (Pin_1)
- net at A4A9A1A1.J2 (OUTPUT): now also ~.1 (Pin_1)
- net at A4A9A1A1.JOY1 (TDC): now also ~.1 (Pin_1)
- net at 4A9A1.J5 (OUTB_GRIP): now also ~.1 (Pin_1)
- net at 4A1W5.1 (Pin_1): now also ~.1 (Pin_1)
- net at 4A1W8.1 (Pin_1): now also ~.1 (Pin_1)
- net at 4A1W10.1 (Pin_1): now also ~.1 (Pin_1)
- net at 4A1W13.1 (Pin_1): now also ~.1 (Pin_1)
- net at 4A1W14.1 (Pin_1): now also ~.1 (Pin_1)
- net at 4A1W17.1 (Pin_1): now also ~.1 (Pin_1)
- net at 4A1W21.1 (Pin_1): now also ~.1 (Pin_1)
- net at 4A1W22.1 (Pin_1): now also ~.1 (Pin_1)
- net at 4A1A.J1 (POWER): now also ~.1 (Pin_1)
- net at 4A1A.USB: now also ~.1 (Pin_1)
- net at 4A13A1W2.1 (Pin_1): now also ~.1 (Pin_1)
- net at 4A11.1 (USB_3.0_A_Type): now also ~.1 (Pin_1)
- net at 4A2A1.USB: now also 4A2A1~.1 (Pin_1)
- net at 4A9A1.USB: now also 4A2A1~.1 (Pin_1)
- net at 4A1W4.1 (Pin_1): now also ~.1 (Pin_1)
- net at 4A1W18.1 (Pin_1): now also ~.1 (Pin_1)
- new net: 4A5A2A1.1 (GND), 4A5A2A1.2 (~D6/A7) (x3)
- new net: 4A5A2A1.2 (~D6/A7), 4A5A2A1.3 (~D3)
- new net: 4A2A1A1.1 (GND), 4A2A1A1.2 (~D6/A7) (x2)
- new net: 4A3A1A1.1 (GND), 4A3A1A1.2 (~D6/A7) (x3)
- new net: 4A3A1A1.2 (~D6/A7), 4A3A1A1.3 (~D3)
- new net: 4A5A1A1.1 (GND), 4A5A1A1.2 (~D6/A7) (x2)

Commit message: UIP Interconnect WIP
UIP Interconnect is WIP
Parts:
- removed (0AxAxWx): ABSIS-CA-C-XXX, symbol Connector_Generic:Conn_01x01
- removed (0AxAxWx): USB A TO B, symbol Connector_Generic:Conn_01x01
- removed (0AxAxWx) (x2): ABSIS-CA-B-XXX, symbol Connector_Generic:Conn_01x01
- removed 4A1W1P? (x2), 4A2A1~ (x11), ~ (x30): ~, symbol Connector_Generic:Conn_01x01
- removed 4A6A1A2: APU BL, symbol ABSIS_2.0:ABSIS_Generic_BackLightPCB
- removed 4A6A1A2: FCS BL, symbol ABSIS_2.0:ABSIS_Generic_BackLightPCB
- removed ~ (x2): ~, symbol Connector:AudioJack2
- added (0AxAxWx): ABSIS-CA-C-XXX, symbol Connector_Generic:Conn_01x01
- added (0AxAxWx): USB A TO B, symbol Connector_Generic:Conn_01x01
- added (0AxAxWx) (x2): ABSIS-CA-B-XXX, symbol Connector_Generic:Conn_01x01
- added 4A1W1P? (x2), 4A2A1~ (x11), ~ (x30): ~, symbol Connector_Generic:Conn_01x01
- added 4A6A1A2: APU BL, symbol ABSIS_2.0:ABSIS_Generic_BackLightPCB
- added 4A6A1A2: FCS BL, symbol ABSIS_2.0:ABSIS_Generic_BackLightPCB
- added ~ (x2): ~, symbol Connector:AudioJack2
Connections:
- net LC<>ABSIS_PSU_PWR: now also (0AxAxWx).1 (Pin_1)
- net LC<>BL1: now also (0AxAxWx).1 (Pin_1)
- net LC<>BL2: now also (0AxAxWx).1 (Pin_1)
- net LC<>UIP_USB_HUB: now also (0AxAxWx).1 (Pin_1)
- net at 4A14A1W2.1 (Pin_1): now also 4A1W1P?.1 (Pin_1)
- net at 4A3A1.USB: now also 4A2A1~.1 (Pin_1)
- net at A4A9A1A1.COM1 (COMM_SW): now also ~.1 (Pin_1)
- net at 4A6A1.USB: now also 4A2A1~.1 (Pin_1)
- net at 4A2A1A2.J2 (BLC_OUT): now also ~.1 (Pin_1)
- net at 4A13A1W8.1 (Pin_1): now also ~.1 (Pin_1)
- net at 4A7A4A2.J2 (BLC_OUT): now also 4A2A1~.1 (Pin_1)
- net at 4A4A3A2.J1 (BLC_IN): now also ~.1 (Pin_1)
- net at 4A7A2A2.J2 (BLC_OUT): now also 4A2A1~.1 (Pin_1)
- net at 4A1W12.1 (Pin_1): now also ~.1 (Pin_1)
- net at 4A9A1.J5 (OUTB_GRIP): now also ~.1 (Pin_1)
- net at 4A1W2.1 (Pin_1): now also ~.1 (Pin_1)
- net at 4A1W14.1 (Pin_1): now also ~.1 (Pin_1)
- net at 4A1W22.1 (Pin_1): now also ~.1 (Pin_1)
- net at 4A5A1.USB: now also 4A2A1~.1 (Pin_1)
- net at 4A13A1W2.1 (Pin_1): now also ~.1 (Pin_1)
- net at 4A1A.J1 (POWER): now also ~.1 (Pin_1)
- net at A4A9A1A1.JOY1 (TDC): now also ~.1 (Pin_1)
- net at A4A9A1A1.ANT1 (ANT_ELEV): now also ~.1 (Pin_1)
- net at 4A9A1.USB: now also 4A2A1~.1 (Pin_1)
- net at 4A2A1~.1 (Pin_1): now also 4A6A1A2.J1 (BLC_IN)
- net at 4A2A1~.1 (Pin_1): now also 4A6A1A2.J2 (BLC_OUT)
- net at 4A6A2A2.J1 (BLC_IN): now also 4A2A1~.1 (Pin_1)
- net at 4A1W8.1 (Pin_1): now also ~.1 (Pin_1)
- net at 4A1W15.1 (Pin_1): now also ~.1 (Pin_1)
- net at 10A1A1A2.J2 (BLC_OUT): now also ~.1 (Pin_1)
- net at 4A1W18.1 (Pin_1): now also ~.1 (Pin_1)
- net at 4A13A1W3.1 (Pin_1): now also ~.1 (Pin_1)
- net at 4A9A1.J9 (IDLE_DET): now also ~.1 (Pin_1)
- net at 4A13A1W4.1 (Pin_1): now also ~.1 (Pin_1)
- net at 4A3A3.USB: now also 4A2A1~.1 (Pin_1)
- net at 4A7A4A2.J1 (BLC_IN): now also 4A2A1~.1 (Pin_1)
- net at 4A11.2 (+5VDC): now also ~.S
- net at 4A11.3 (GND): now also ~.T
- net at 4A9A1.J10 (MAX_DET): now also ~.1 (Pin_1)
- net at 4A4A1A2.J1 (BLC_IN): now also ~.1 (Pin_1)
- net at 4A4A2A2.J2 (BLC_OUT): now also ~.1 (Pin_1)
- net at A4A9A1A1.CAGE1 (CAGE): now also ~.1 (Pin_1)
- net at 4A1W16.1 (Pin_1): now also ~.1 (Pin_1)
- net at 4A1W20.1 (Pin_1): now also ~.1 (Pin_1)
- net at 4A14A1W1.1 (Pin_1): now also 4A1W1P?.1 (Pin_1)
- net at 4A9A1.J7 (OUTB_LIMIT): now also ~.1 (Pin_1)
- net at 4A9A1.J4 (INB_GRIP): now also ~.1 (Pin_1)
- net at 4A9A1.J6 (INB_LIMIT): now also ~.1 (Pin_1)
- net at 4A1W3.1 (Pin_1): now also ~.1 (Pin_1)
- new net: 4A3A1A1.1 (GND), 4A3A1A1.2 (~D6/A7) (x3)
- new net: 4A3A1A1.2 (~D6/A7), 4A3A1A1.3 (~D3)
- new net: 4A12.~ (USB_OUT), ~.S
- new net: 4A12.~ (USB_OUT), ~.T
- new net: 4A5A1A1.1 (GND), 4A5A1A1.2 (~D6/A7) (x2)
- new net: 4A5A2A1.1 (GND), 4A5A2A1.2 (~D6/A7) (x3)
- new net: 4A5A2A1.2 (~D6/A7), 4A5A2A1.3 (~D3)
- new net: 4A2A1~.1 (Pin_1), 4A6A1A2.J2 (BLC_OUT)
- new net: 4A2A1A1.1 (GND), 4A2A1A1.2 (~D6/A7) (x2)
- new net: 4A2A1~.1 (Pin_1), 4A6A1A2.J1 (BLC_IN)

Commit message: Made all interfaces USB 3.0 compatible.
All interfaces USB 3.0 compatible.
Closes #466
Parts:
- removed 4A12: HB-U14P, symbol OpenHornet:HB-U14P
- removed 4A13A1W9: USB A TO A EXTENSION, symbol Connector_Generic:Conn_01x01
- removed 4A1W11P3, 4A1W1P?, ~ (x2): ~, symbol Connector_Generic:Conn_01x01
- removed 4A1W29: USB A TO A, symbol Connector_Generic:Conn_01x01
- removed 4A1W31: USB A EXTENSION, symbol Connector_Generic:Conn_01x01
- removed ~: ~, symbol Connector:AudioJack2
- added (4A13A1W1): (1681-02C), symbol Connector_Generic:Conn_01x01
- added 4A11A2, 4A11A3, 4A11A4: B09V6WY1SD, symbol OpenHornet:B09V6WY1SD
- added 4A1W11P3, 4A1W11P4, 4A1W11P5: PP-002D-01, symbol OpenHornet:Barrel_Plug
- added ~ (x3): ~, symbol Connector:Barrel_Jack
- added ~?: ~, symbol Connector_Generic:Conn_01x01
- 4A13A1W1: value 1587-02C -> 1681-02C
- 4A1W11: value ABSIS-CA-A-XXX -> ABSIS-CA-A-XXX ***MODIFIED***
- renumbered 4A11 to 4A11A1, 4A1W30 to 4A13A1W1
Connections:
- net 3A3A1_USB: now also 4A14A1W1.1 (Pin_1), 4A11A3.~ (USB_OUT)
- net 4A12_USB: now also 4A13A1W1.1 (Pin_1), (4A13A1W1).1 (Pin_1)
- net 4A1A_USB: now also 4A11A2.~ (USB_OUT)
- net 4A2A1_USB: now also 4A11A2.~ (USB_OUT)
- net 4A3A1_USB: now also 4A11A2.~ (USB_OUT)
- net 4A3A3_USB: now also 4A11A2.~ (USB_OUT)
- net 4A5A1_USB: now also 4A11A3.~ (USB_OUT)
- net 4A5A2_USB: now also 4A11A2.~ (USB_OUT)
- net 4A6A1_USB: now also 4A11A3.~ (USB_OUT)
- net 4A9A1_USB: now also 4A11A3.~ (USB_OUT)
- net 4A11_USB renamed 4A11A1_USB
- net 4A11A1_USB: now also 4A11A3.~ (USB_OUT)
- new net: 4A3A1A1.1 (GND), 4A3A1A1.2 (~D6/A7) (x3)
- new net: 4A3A1A1.2 (~D6/A7), 4A3A1A1.3 (~D3)
- new net: 4A5A1A1.1 (GND), 4A5A1A1.2 (~D6/A7) (x2)
- new net: 4A5A2A1.1 (GND), 4A5A2A1.2 (~D6/A7) (x3)
- new net: 4A5A2A1.2 (~D6/A7), 4A5A2A1.3 (~D3)
- new net: 4A2A1A1.1 (GND), 4A2A1A1.2 (~D6/A7) (x2)
- new net: 4A11A2.~ (USB_OUT), ~.1
- new net: 4A11A2.~ (USB_OUT), ~.2
- new net: 4A11A2.~ (USB_OUT), ~?.1 (Pin_1)
- new net: 4A11A3.~ (USB_OUT), ~.1
- new net: 4A11A3.~ (USB_OUT), ~.2
- new net: 4A11A4.~ (USB_OUT), ~.1
- new net: 4A11A4.~ (USB_OUT), ~.2
- new net +5V: 4A1W11P3.1, 4A1W11P4.1, 4A1W11P5.1
- new net 4A11A3_USB: 4A11A2.~ (USB_OUT), 4A11A3.~ (USB_OUT)
- new net 4A11A4_USB: 4A11A3.~ (USB_OUT), 4A11A4.~ (USB_OUT)
- new net GND: 4A1W11P3.2, 4A1W11P4.2, 4A1W11P5.2
- no-connect marks 294 -> 291
Other:
- note added: "(4A1W11)"
- note added: "(ABSIS-CA-A-XXX ***MODIFIED***)"
- note added: "***4A1W11 MODIFIED***\n+5V/GND LINES ONLY\nREMOVE SECOND CONNECTOR\nTERMINATE WITH SPLICED OEM \n CONNECTOR TO CREATE P2\nTERMINATE P3/P4/P5 AS SHOWN"
- note added: "4-PRT USB HUB"
- note added: "APU, ETC"
- note added: "BRK GAUGE, ETC"
- note added: "CENTER TUB"
- note added: "EXT LTS, ETC"
- note added: "FUTURE EXP"
- note added: "LC HID MASTER"
- note added: "LC USB HUB #2"
- note added: "LC USB HUB #3"
- note added: "LDG GEAR PANEL"
- note added: "OBOGS"
- note added: "SELECT JETT"
- note added: "USB HUBS"
- note removed: "***4A1W11 MODIFIED***\n+5V/GND LINES ONLY\nREMOVE SECOND CONNECTOR\nTERMINATE WITH SPLICED OEM \n CONNECTOR TO CREATE P2/P3"
