File: ECAD/PCBs/ABSIS/ABSIS_ATX_PSU_Board/ATX_PSU_Board.sch (KiCad schematic (older format))
At the start: 22 parts, among them J1 Power Swtich, J10 MEGA BUS POWER, J2 ATX-24, J3 ABSIS BACKLIGHT PWR, J4 MEGA BUS POWER, J5 MEGA BUS POWER, J6 MEGA BUS POWER, J7 MEGA BUS POWER, J8 MEGA BUS POWER, J9 MEGA BUS POWER

Commit message: Small tweaks
Removed unused digikey lib
deleted separate PTH and TH DRL files and combined into single file IAW JLCPCB requirements
Moved to direct subfolder (removed extra folder layer.)
Parts:
- J2: symbol Connector:ATX-24 -> ATX_PSU_Board-rescue:ATX-24-Connector
Changed lines of the file:
@@
 EESchema Schematic File Version 4
+LIBS:ATX_PSU_Board-cache
 EELAYER 30 0
 EELAYER END
@@
 NoConn ~ 3000 2200
 $Comp
-L Connector:ATX-24 J2
+L ATX_PSU_Board-rescue:ATX-24-Connector J2
 U 1 1 5FA8791F
 P 2500 1800

Commit message: ABSIS ATX PSU Board Update
Added - 1x ABSIS Master connector
Added - 8x 5V accessory 1x2 connector
Added - 5x 12V accessory 1x2 connector
Added - PWR-OK LED
Added - External 5V input XT60 connector for use with Mean well PSU if required
Added - External 12V input XT60 connector for use with Mean well PSU if required.
Added - ButtKicker amp XT60 connector
Added - Silkscreen stating ButtKicker amp is 12V on back.
Added - Extensive silkscreening of pins
Changed - Connector locations to maximize PCB space.
Changed - 5V from internal layer 2 to back layer to allow 2oz copper vs 0.5oz copper fill for the high current backlighting.
Changed - 3.3V from back layer to internal layer 2, high current not required, 0.5oz copper fill will be plenty.
Removed - CC-BY-NC-SA logo from front silkscreen due to lack of space.
Parts:
- added D5: Green LED, LED_SMD:LED_0603_1608Metric_Pad1.05x0.95mm_HandSolder, symbol Device:LED
- added J11: MEGA BUS 8, Connector_Molex:Molex_Mini-Fit_Jr_5566-08A2_2x04_P4.20mm_Vertical, symbol Connector_Generic:Conn_02x04_Top_Bottom
- added J12: 5V Accessory 1, Connector_Molex:Molex_Mini-Fit_Jr_5566-02A_2x01_P4.20mm_Vertical, symbol Connector:Conn_01x02_Female
- added J13: 5V Accessory 2, Connector_Molex:Molex_Mini-Fit_Jr_5566-02A_2x01_P4.20mm_Vertical, symbol Connector:Conn_01x02_Female
- added J14: 5V Accessory 3, Connector_Molex:Molex_Mini-Fit_Jr_5566-02A_2x01_P4.20mm_Vertical, symbol Connector:Conn_01x02_Female
- added J15: 5V Accessory 4, Connector_Molex:Molex_Mini-Fit_Jr_5566-02A_2x01_P4.20mm_Vertical, symbol Connector:Conn_01x02_Female
- added J16: 5V Accessory 5, Connector_Molex:Molex_Mini-Fit_Jr_5566-02A_2x01_P4.20mm_Vertical, symbol Connector:Conn_01x02_Female
- added J17: 5V Accessory 6, Connector_Molex:Molex_Mini-Fit_Jr_5566-02A_2x01_P4.20mm_Vertical, symbol Connector:Conn_01x02_Female
- added J18: 5V Accessory 7, Connector_Molex:Molex_Mini-Fit_Jr_5566-02A_2x01_P4.20mm_Vertical, symbol Connector:Conn_01x02_Female
- added J19: 5V Accessory 8, Connector_Molex:Molex_Mini-Fit_Jr_5566-02A_2x01_P4.20mm_Vertical, symbol Connector:Conn_01x02_Female
- added J20: 12V Accessory 1, Connector_Molex:Molex_Mini-Fit_Jr_5566-02A_2x01_P4.20mm_Vertical, symbol Connector:Conn_01x02_Female
- added J21: 12V Accessory 2, Connector_Molex:Molex_Mini-Fit_Jr_5566-02A_2x01_P4.20mm_Vertical, symbol Connector:Conn_01x02_Female
- added J22: 12V Accessory 3, Connector_Molex:Molex_Mini-Fit_Jr_5566-02A_2x01_P4.20mm_Vertical, symbol Connector:Conn_01x02_Female
- added J23: 12V Accessory 4, Connector_Molex:Molex_Mini-Fit_Jr_5566-02A_2x01_P4.20mm_Vertical, symbol Connector:Conn_01x02_Female
- added J24: 12V Accessory 5, Connector_Molex:Molex_Mini-Fit_Jr_5566-02A_2x01_P4.20mm_Vertical, symbol Connector:Conn_01x02_Female
- added J28: EXTERNAL 5V IN, Connector_AMASS:AMASS_XT60-M_1x02_P7.20mm_Vertical, symbol Connector:Conn_01x02_Female
- added J29: BUTTKICKER AMP, Connector_AMASS:AMASS_XT60-F_1x02_P7.20mm_Vertical, symbol Connector:Conn_01x02_Female
- added J30: EXTERNAL 12V IN, Connector_AMASS:AMASS_XT60-M_1x02_P7.20mm_Vertical, symbol Connector:Conn_01x02_Female
- added R5: 150, Resistor_SMD:R_0603_1608Metric_Pad0.98x0.95mm_HandSolder, symbol Device:R
- D1: value Green LED -> Blue LED
- J1: value Power Swtich -> POWER SWITCH
- J10: renamed from J9; value MEGA BUS POWER -> MEGA BUS 7
- J3: value ABSIS BACKLIGHT PWR -> ABSIS BACKLIGHT
- J4: value MEGA BUS POWER -> MEGA BUS 1
- J5: value MEGA BUS POWER -> MEGA BUS 2
- J6: value MEGA BUS POWER -> MEGA BUS 3
- J7: renamed from J10; value MEGA BUS POWER -> MEGA BUS 4
- J8: renamed from J7; value MEGA BUS POWER -> MEGA BUS 5
- J9: renamed from J8; value MEGA BUS POWER -> MEGA BUS 6
Connections:
- wire segments 57 -> 64
- no-connect marks 2 -> 1
Other:
- note added: "Accessory Connectors"

Commit message: ABSIS ATX Power Distro Board Update
Added - Exposed traces on back for high current 12 and 5V devices if needed to be filled with solder.
Added - 2 PCIE 6 pin headers for additional 12v supply.
Changed - Position of connectors to create a high current 12V island
Added - 12V partial copper fill on 5V back plane to give it 2oz copper not 0.5oz internal for high current devices.
Changed - CC-BY-NC-SA logo to text form, not enough space to keep it.
Changed - Board is now 10mm longer.
Changed - Various silkscreen label positions.
Changed - Revision from 2 to 3
Changed - Manufacturing files to match changes.
Parts:
- added J25: PCIE IN 2, Connector_Molex:Molex_Mini-Fit_Jr_5566-06A_2x03_P4.20mm_Vertical, symbol Connector_Generic:Conn_02x03_Top_Bottom
- added J26: PCIE IN 1, Connector_Molex:Molex_Mini-Fit_Jr_5566-06A_2x03_P4.20mm_Vertical, symbol Connector_Generic:Conn_02x03_Top_Bottom
- D1, D2, D3, D4, D5: symbol Device:LED -> ATX_PSU_Board-rescue:LED-Device
- H1, H2, H3, H4: symbol Mechanical:MountingHole -> ATX_PSU_Board-rescue:MountingHole-Mechanical
- J1: symbol Connector_Generic:Conn_01x02 -> ATX_PSU_Board-rescue:Conn_01x02-Connector_Generic
- J10, J11, J4, J5, J6, J7, J8, J9: symbol Connector_Generic:Conn_02x04_Top_Bottom -> ATX_PSU_Board-rescue:Conn_02x04_Top_Bottom-Connector_Generic
- J12, J13, J14, J15, J16, J17, J18, J19, J20, J21, J22, J23, J24, J28, J29, J30: symbol Connector:Conn_01x02_Female -> ATX_PSU_Board-rescue:Conn_01x02_Female-Connector
- J3: symbol Connector_Generic:Conn_02x05_Top_Bottom -> ATX_PSU_Board-rescue:Conn_02x05_Top_Bottom-Connector_Generic
- R1, R2, R3, R4, R5: symbol Device:R -> ATX_PSU_Board-rescue:R-Device
Connections:
- wire segments 64 -> 74

Commit message: ATX PSU Breakout Rev 4
Expanded PS_ON Header to include +5VSB and PWR_OK Pins.
Parts:
- J1: value POWER SWITCH -> I/O; footprint Connector_PinHeader_2.54mm:PinHeader_1x02_P2.54mm_Vertical -> Connector_PinHeader_2.54mm:PinHeader_1x04_P2.54mm_Vertical; symbol ATX_PSU_Board-rescue:Conn_01x02-Connector_Generic -> Connector_Generic:Conn_01x04
Connections:
- net +5VSB_SUPPLY: now also J1.2 (Pin_2)
- net GND: now also J1.4 (Pin_4); no longer J1.2 (Pin_2)
- net PWR_OK: now also J1.3 (Pin_3)
Other:
- note added: "CONNECTION TO PIT MANAGER"
- note removed: "CONNECTION TO POWER SWITCH PANEL"
Changed lines of the file:
@@
 	1650 1400 2000 1400
 $Comp
-L ATX_PSU_Board-rescue:Conn_01x02-Connector_Generic J1
+L Connector_Generic:Conn_01x04 J1
 U 1 1 5FA8D26E
 P 8800 5250
 F 0 "J1" H 8880 5242 50  0000 L CNN
-F 1 "POWER SWITCH" H 8880 5151 50  0000 L CNN
-F 2 "Connector_PinHeader_2.54mm:PinHeader_1x02_P2.54mm_Vertical" H 8800 5250 50  0001 C CNN
+F 1 "I/O" H 8880 5151 50  0000 L CNN
+F 2 "Connector_PinHeader_2.54mm:PinHeader_1x04_P2.54mm_Vertical" H 8800 5250 50  0001 C CNN
 F 3 "~" H 8800 5250 50  0001 C CNN
 	1    8800 5250
@@
 $EndComp
 Wire Wire Line
-	8500 5450 8500 5350
-Wire Wire Line
-	8500 5350 8600 5350
-Text Label 8250 5250 0    50   ~ 0
-PS_ON
-Wire Wire Line
-	8600 5250 8250 5250
+	8500 5450 8600 5450
 $Comp
 L ATX_PSU_Board-rescue:Conn_02x04_Top_Bottom-Connector_Generic J4
@@
 NOTE: LED Feedback is optional and not required
 Text Notes 8250 5000 0    39   ~ 0
-CONNECTION TO POWER SWITCH PANEL
+CONNECTION TO PIT MANAGER
 Wire Notes Line
 	8200 4850 9450 4850
@@
 Wire Wire Line
 	2800 4050 2800 4150
+Text Label 8600 5250 2    31   ~ 0
++5VSB_SUPPLY
+Text Label 8600 5350 2    31   ~ 0
+PWR_OK
+Text Label 8600 5150 2    50   ~ 0
+PS_ON
 $EndSCHEMATC

Commit message: ABSIS ATX PSU PCB Update
Changed - SMD indicator LEDs and Resistors to THT. Reason: To decrease cost of manufacture without needing SMT assembly.
Parts:
- D1, D2, D3, D4, D5: footprint LED_SMD:LED_0603_1608Metric_Pad1.05x0.95mm_HandSolder -> LED_THT:LED_D3.0mm
- R1, R2, R3, R4, R5: footprint Resistor_SMD:R_0603_1608Metric_Pad0.98x0.95mm_HandSolder -> Resistor_THT:R_Axial_DIN0207_L6.3mm_D2.5mm_P7.62mm_Horizontal
Changed lines of the file:
@@
 F 0 "R1" V 9100 1200 50  0000 C CNN
 F 1 "150" V 9200 1200 50  0000 C CNN
-F 2 "Resistor_SMD:R_0603_1608Metric_Pad0.98x0.95mm_HandSolder" V 9130 1200 50  0001 C CNN
+F 2 "Resistor_THT:R_Axial_DIN0207_L6.3mm_D2.5mm_P7.62mm_Horizontal" V 9130 1200 50  0001 C CNN
 F 3 "https://datasheet.lcsc.com/szlcsc/1811081724_UNI-ROYAL-Uniroyal-Elec-0603WAF1500T5E_C22808.pdf" H 9200 1200 50  0001 C CNN
 F 4 "C22808" V 9200 1200 50  0001 C CNN "LCSC"
@@
 F 0 "D1" H 9500 1250 39  0000 C CNN
 F 1 "Blue LED" H 9750 1100 39  0000 C CNN
-F 2 "LED_SMD:LED_0603_1608Metric_Pad1.05x0.95mm_HandSolder" H 9850 1400 60  0001 L CNN
+F 2 "LED_THT:LED_D3.0mm" H 9850 1400 60  0001 L CNN
 F 3 "https://datasheet.lcsc.com/szlcsc/Foshan-NationStar-Optoelectronics-FC-DA1608UGK-520D10_C84267.pdf" H 9850 1500 60  0001 L CNN
 F 4 "Optoelectronics" H 9850 1800 60  0001 L CNN "Category"
@@
 F 0 "R2" V 9100 1500 50  0000 C CNN
 F 1 "150" V 9200 1500 50  0000 C CNN
-F 2 "Resistor_SMD:R_0603_1608Metric_Pad0.98x0.95mm_HandSolder" V 9130 1500 50  0001 C CNN
+F 2 "Resistor_THT:R_Axial_DIN0207_L6.3mm_D2.5mm_P7.62mm_Horizontal" V 9130 1500 50  0001 C CNN
 F 3 "https://datasheet.lcsc.com/szlcsc/1811081724_UNI-ROYAL-Uniroyal-Elec-0603WAF1500T5E_C22808.pdf" H 9200 1500 50  0001 C CNN
 F 4 "C22808" V 9200 1500 50  0001 C CNN "LCSC"
@@
 F 0 "R3" V 9100 1800 50  0000 C CNN
 F 1 "56" V 9200 1800 50  0000 C CNN
-F 2 "Resistor_SMD:R_0603_1608Metric_Pad0.98x0.95mm_HandSolder" V 9130 1800 50  0001 C CNN
+F 2 "Resistor_THT:R_Axial_DIN0207_L6.3mm_D2.5mm_P7.62mm_Horizontal" V 9130 1800 50  0001 C CNN
 F 3 "https://datasheet.lcsc.com/szlcsc/1811081724_UNI-ROYAL-Uniroyal-Elec-0603WAF560JT5E_C25196.pdf" H 9200 1800 50  0001 C CNN
 F 4 "C25196" V 9200 1800 50  0001 C CNN "LCSC"
@@
 F 0 "R4" V 9100 2100 50  0000 C CNN
 F 1 "560" V 9200 2100 50  0000 C CNN
-F 2 "Resistor_SMD:R_0603_1608Metric_Pad0.98x0.95mm_HandSolder" V 9130 2100 50  0001 C CNN
+F 2 "Resistor_THT:R_Axial_DIN0207_L6.3mm_D2.5mm_P7.62mm_Horizontal" V 9130 2100 50  0001 C CNN
 F 3 "https://datasheet.lcsc.com/szlcsc/1811021213_UNI-ROYAL-Uniroyal-Elec-0603WAF5600T5E_C23204.pdf" H 9200 2100 50  0001 C CNN
 F 4 "C23204" V 9200 2100 50  0001 C CNN "LCSC"
@@
 F 0 "D2" H 9500 1550 39  0000 C CNN
 F 1 "Green LED" H 9750 1400 39  0000 C CNN
-F 2 "LED_SMD:LED_0603_1608Metric_Pad1.05x0.95mm_HandSolder" H 9850 1700 60  0001 L CNN
+F 2 "LED_THT:LED_D3.0mm" H 9850 1700 60  0001 L CNN
 F 3 "https://datasheet.lcsc.com/szlcsc/Foshan-NationStar-Optoelectronics-FC-DA1608UGK-520D10_C84267.pdf" H 9850 1800 60  0001 L CNN
 F 4 "Optoelectronics" H 9850 2100 60  0001 L CNN "Category"
@@
 F 0 "D3" H 9500 1850 39  0000 C CNN
 F 1 "Green LED" H 9750 1700 39  0000 C CNN
-F 2 "LED_SMD:LED_0603_1608Metric_Pad1.05x0.95mm_HandSolder" H 9850 2000 60  0001 L CNN
+F 2 "LED_THT:LED_D3.0mm" H 9850 2000 60  0001 L CNN
 F 3 "https://datasheet.lcsc.com/szlcsc/Foshan-NationStar-Optoelectronics-FC-DA1608UGK-520D10_C84267.pdf" H 9850 2100 60  0001 L CNN
 F 4 "Optoelectronics" H 9850 2400 60  0001 L CNN "Category"
@@
 F 0 "D4" H 9500 2150 39  0000 C CNN
 F 1 "Green LED" H 9750 2000 39  0000 C CNN
-F 2 "LED_SMD:LED_0603_1608Metric_Pad1.05x0.95mm_HandSolder" H 9850 2300 60  0001 L CNN
+F 2 "LED_THT:LED_D3.0mm" H 9850 2300 60  0001 L CNN
 F 3 "https://datasheet.lcsc.com/szlcsc/Foshan-NationStar-Optoelectronics-FC-DA1608UGK-520D10_C84267.pdf" H 9850 2400 60  0001 L CNN
 F 4 "LED GREEN DIFFUSED" H 9850 3100 60  0001 L CNN "Description"
@@
 F 0 "R5" V 9100 2400 50  0000 C CNN
 F 1 "150" V 9200 2400 50  0000 C CNN
-F 2 "Resistor_SMD:R_0603_1608Metric_Pad0.98x0.95mm_HandSolder" V 9130 2400 50  0001 C CNN
+F 2 "Resistor_THT:R_Axial_DIN0207_L6.3mm_D2.5mm_P7.62mm_Horizontal" V 9130 2400 50  0001 C CNN
 F 3 "https://datasheet.lcsc.com/szlcsc/1811021213_UNI-ROYAL-Uniroyal-Elec-0603WAF5600T5E_C23204.pdf" H 9200 2400 50  0001 C CNN
 F 4 "C23204" V 9200 2400 50  0001 C CNN "LCSC"
@@
 F 0 "D5" H 9500 2450 39  0000 C CNN
 F 1 "Green LED" H 9750 2300 39  0000 C CNN
-F 2 "LED_SMD:LED_0603_1608Metric_Pad1.05x0.95mm_HandSolder" H 9850 2600 60  0001 L CNN
+F 2 "LED_THT:LED_D3.0mm" H 9850 2600 60  0001 L CNN
 F 3 "https://datasheet.lcsc.com/szlcsc/Foshan-NationStar-Optoelectronics-FC-DA1608UGK-520D10_C84267.pdf" H 9850 2700 60  0001 L CNN
 F 4 "LED GREEN DIFFUSED" H 9850 3400 60  0001 L CNN "Description"

Commit message: ATX PSU Schematic Documentation
Added - Notes to many connectors explaining their use.
Added - Note stating it is a 4 layer board.
Changed - Layout of schematic into input and output sections for easier understanding at a glance.
Changed - Indicator LED resistor values to limit current to ~2mA to match arduino indicator brightness. Previous values made them 10-20mA.
Parts:
- removed J13: 5V Accessory 2, Connector_Molex:Molex_Mini-Fit_Jr_5566-02A_2x01_P4.20mm_Vertical, symbol ATX_PSU_Board-rescue:Conn_01x02_Female-Connector
- removed J14: 5V Accessory 3, Connector_Molex:Molex_Mini-Fit_Jr_5566-02A_2x01_P4.20mm_Vertical, symbol ATX_PSU_Board-rescue:Conn_01x02_Female-Connector
- removed J15: 5V Accessory 4, Connector_Molex:Molex_Mini-Fit_Jr_5566-02A_2x01_P4.20mm_Vertical, symbol ATX_PSU_Board-rescue:Conn_01x02_Female-Connector
- removed J16: 5V Accessory 5, Connector_Molex:Molex_Mini-Fit_Jr_5566-02A_2x01_P4.20mm_Vertical, symbol ATX_PSU_Board-rescue:Conn_01x02_Female-Connector
- removed J17: 5V Accessory 6, Connector_Molex:Molex_Mini-Fit_Jr_5566-02A_2x01_P4.20mm_Vertical, symbol ATX_PSU_Board-rescue:Conn_01x02_Female-Connector
- removed J18: 5V Accessory 7, Connector_Molex:Molex_Mini-Fit_Jr_5566-02A_2x01_P4.20mm_Vertical, symbol ATX_PSU_Board-rescue:Conn_01x02_Female-Connector
- removed J19: 5V Accessory 8, Connector_Molex:Molex_Mini-Fit_Jr_5566-02A_2x01_P4.20mm_Vertical, symbol ATX_PSU_Board-rescue:Conn_01x02_Female-Connector
- removed J20: 12V Accessory 1, Connector_Molex:Molex_Mini-Fit_Jr_5566-02A_2x01_P4.20mm_Vertical, symbol ATX_PSU_Board-rescue:Conn_01x02_Female-Connector
- removed J21: 12V Accessory 2, Connector_Molex:Molex_Mini-Fit_Jr_5566-02A_2x01_P4.20mm_Vertical, symbol ATX_PSU_Board-rescue:Conn_01x02_Female-Connector
- removed J22: 12V Accessory 3, Connector_Molex:Molex_Mini-Fit_Jr_5566-02A_2x01_P4.20mm_Vertical, symbol ATX_PSU_Board-rescue:Conn_01x02_Female-Connector
- removed J23: 12V Accessory 4, Connector_Molex:Molex_Mini-Fit_Jr_5566-02A_2x01_P4.20mm_Vertical, symbol ATX_PSU_Board-rescue:Conn_01x02_Female-Connector
- removed J24: 12V Accessory 5, Connector_Molex:Molex_Mini-Fit_Jr_5566-02A_2x01_P4.20mm_Vertical, symbol ATX_PSU_Board-rescue:Conn_01x02_Female-Connector
- added J13: 5V Accessory 2, Connector_Molex:Molex_Mini-Fit_Jr_5566-02A_2x01_P4.20mm_Vertical, symbol ATX_PSU_Board-rescue:Conn_01x02-Connector_Generic
- added J14: 5V Accessory 3, Connector_Molex:Molex_Mini-Fit_Jr_5566-02A_2x01_P4.20mm_Vertical, symbol ATX_PSU_Board-rescue:Conn_01x02-Connector_Generic
- added J15: 5V Accessory 4, Connector_Molex:Molex_Mini-Fit_Jr_5566-02A_2x01_P4.20mm_Vertical, symbol ATX_PSU_Board-rescue:Conn_01x02-Connector_Generic
- added J16: 5V Accessory 5, Connector_Molex:Molex_Mini-Fit_Jr_5566-02A_2x01_P4.20mm_Vertical, symbol ATX_PSU_Board-rescue:Conn_01x02-Connector_Generic
- added J17: 5V Accessory 6, Connector_Molex:Molex_Mini-Fit_Jr_5566-02A_2x01_P4.20mm_Vertical, symbol ATX_PSU_Board-rescue:Conn_01x02-Connector_Generic
- added J18: 5V Accessory 7, Connector_Molex:Molex_Mini-Fit_Jr_5566-02A_2x01_P4.20mm_Vertical, symbol ATX_PSU_Board-rescue:Conn_01x02-Connector_Generic
- added J19: 5V Accessory 8, Connector_Molex:Molex_Mini-Fit_Jr_5566-02A_2x01_P4.20mm_Vertical, symbol ATX_PSU_Board-rescue:Conn_01x02-Connector_Generic
- added J20: 12V Accessory 1, Connector_Molex:Molex_Mini-Fit_Jr_5566-02A_2x01_P4.20mm_Vertical, symbol ATX_PSU_Board-rescue:Conn_01x02-Connector_Generic
- added J21: 12V Accessory 2, Connector_Molex:Molex_Mini-Fit_Jr_5566-02A_2x01_P4.20mm_Vertical, symbol ATX_PSU_Board-rescue:Conn_01x02-Connector_Generic
- added J22: 12V Accessory 3, Connector_Molex:Molex_Mini-Fit_Jr_5566-02A_2x01_P4.20mm_Vertical, symbol ATX_PSU_Board-rescue:Conn_01x02-Connector_Generic
- added J23: 12V Accessory 4, Connector_Molex:Molex_Mini-Fit_Jr_5566-02A_2x01_P4.20mm_Vertical, symbol ATX_PSU_Board-rescue:Conn_01x02-Connector_Generic
- added J24: 12V Accessory 5, Connector_Molex:Molex_Mini-Fit_Jr_5566-02A_2x01_P4.20mm_Vertical, symbol ATX_PSU_Board-rescue:Conn_01x02-Connector_Generic
- J12, J28, J29, J30: symbol ATX_PSU_Board-rescue:Conn_01x02_Female-Connector -> ATX_PSU_Board-rescue:Conn_01x02-Connector_Generic
- R1: value 150 -> 560
- R2, R5: value 150 -> 1k5
- R3: value 56 -> 560
- R4: value 560 -> 5k1
Connections:
- net +12V_SUPPLY: now also J20.1 (Pin_1), J21.1 (Pin_1), J22.1 (Pin_1), J23.1 (Pin_1), J24.1 (Pin_1)
- net +5V_SUPPLY: now also J13.1 (Pin_1), J14.1 (Pin_1), J15.1 (Pin_1), J16.1 (Pin_1), J17.1 (Pin_1), J18.1 (Pin_1), J19.1 (Pin_1)
- net GND: now also J13.2 (Pin_2), J14.2 (Pin_2), J15.2 (Pin_2), J16.2 (Pin_2), J17.2 (Pin_2), J18.2 (Pin_2), J19.2 (Pin_2), J20.2 (Pin_2), J21.2 (Pin_2), J22.2 (Pin_2), J23.2 (Pin_2), J24.2 (Pin_2)
Other:
- note added: "12V Accessories"
- note added: "5V Accessories"
- note added: "Note: J3 - J24 connectors are to use Molex Mini-Fit Jr"
- note added: "Note: LED Feedback is optional"
- note added: "Note: Optional, used to provide additional 12V capacity from the ATX PSU."
- note added: "Note: This is to be manufactured as a 4 layer PCB"
- note added: "Note: XT60 Connector\nHigh current output to Buttkicker power amplifier"
- note added: "Note: XT60 Male Connector\nIf an ATX PSU is used, this connection should not need to be utilised.\nCan also be used to connect a dedicated 12V PSU if an ATX one is not used."
- note added: "Note: XT60 Male Connector\nMost ATX PSUs provide 20A max @ 5V.\nIf additional 5V capacity is required, this port should be used.\nIt can also be used to connect a dedicated 5V PSU."
- note added: "Note:\nOptional, used to provide additional 12V capacity from the ATX PSU."
- note added: "Note:\nQuality ATX PSU of 650W or greater should be used.\nA modular cable model is recommended.\nMake sure it is rated for 20A @ 5V"
- note added: "Power Sinks"
- note added: "Power Sources"
- note removed: "Accessory Connectors"
- note removed: "NOTE: LED Feedback is optional and not required"
- note removed: "Power Connectors"
- moved on the sheet: D1, D2, D3, D4, D5, H1, H2, H3, H4, J1, J10, J11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
