File: ECAD/PCBs/OH_Specific/Backlighting_Type A/PCB, APU PANEL/PCB, APU PANEL.kicad_pcb (KiCad board)
At the start: 2 copper layers, 48.1 x 115.6 mm, 46 parts, among them J1 Conn_01x04_Female, J2 Conn_01x04_Female

Commit message: Update: || KiCad 5 to 6 transition - APU Panel ||  ECAD Cleanup/Consolidation ||
---------------------------------------
APU PANEL TRANSITION
------------------------------------
0:  Begin naming convention to match OH nomenclature:  - Rename "APU Panel" to "PCB, APU PANEL"

1:  Added "Legacy" folder:  Used to store all files that are no longer being used and are associated with KiCad 5 and older.

2:  Removed old "APU Panel" BOM/CPL files:  Files were from APU Ver.1 that were parsed from a different plugin.  Outdated and no longer needed.

3:  Moved "fp-info-cache" to Legacy.:  "Cache to speed up loading of footprint libraries."  File is excess and not needed.  [Ref.:  https://docs.kicad.org/master/en/kicad/kicad.html

4:  Removed "sym-lib-table":  Legacy, references a file that doesn't currently exist and is no longer needed anyway due to KiCad 6 features.

5:  Updated APU Panel Schematic:  - Fixed component footprint paths; Now point to OH_Footprints library.
-Molex Mini-Fit Jr.
-Generic Capacitor, Resisters, LEDs

6:  Updated APU Panel PCB:   - Fixed Logo footprint paths; now points to OH_Footprints.
-Molex Mini-Fit Jr.
-Generic Capacitor, Resisters, LEDs

***3d model's now properly display for PCB board.

-Added new 3d images of PCB.
-------------------------------------------
Updated ECAD Cleanup/Consolidation
---------------------------------------------------
7:  Renamed "3D" folder to "OH_3dModels"

8:  Added footprint to OH_Footprints library:  Molex_Mini-Fit_Jr_5566-04A_2x02_P4.20mm_Vertical.  - Molex connector is available in Generic KiCad Libraries, but without a 3d Model attached.  Saving a copy within OH libraries allows us to reference a 3D model (which is conveniently already in the 3d model folder of the OH library package).  _Generic KiCad libraries are read-only_

9:  Referenced 3D Model for Molex_Mini-Fit_Jr_5566-04A_2x02_P4.20mm_Vertical within the footprint:  Molex Mini-fit 3D model is already located in ECAD/lib/OH_3DModels.

10:  WS2812B-Min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
Other:
- board text added: "Version 2.3"
- board text removed: "Version 2.2"
