File: ECAD/PCBs/Backlight PCBs/Backlighting_Type A/SIM POWER PANEL/SIM POWER PANEL.kicad_sch (KiCad schematic)
At the start: 77 parts, among them J1 Conn_01x04_Female, J2 Conn_01x04_Female

Commit message: Drawing Sheet & Silkscreen update - Backlight Panels (Fc thru Spin)
1:  Updated/Relinked Drawing Sheet for both PCB and Schematics
2:  Standardized Silkscreen (if required)

Finished Remaining Backlighting Type A & Type B PCBs.....
Other:
- title: (none) -> SIM POWER PANEL
Changed lines of the file:
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@@
 (kicad_sch (version 20211123) (generator eeschema)
   (paper "A4")
+  (title_block
+    (title "SIM POWER PANEL")
+    (date "2023-02-10")
+    (rev "3")
+  )
   (junction (at 29.21 91.44) (diameter 0) (color 0 0 0 0)
   )

Commit message: KiCad 7 Transition - SIM POWER Panel
PCB and Schematic standardization
Updated silkscreen text
Adjusted traces to prevent conflicts
Add Testpoints
Recompiled assets and manufacturing files
Parts:
- removed C1: C_Polarized, OH_Footprints:CP_Elec_8x10, symbol Device:C_Polarized
- removed C10, C11, C12, C13, C14, C15, C16, C17, C18, C19, C2, C20, C21, C22, C23, C24, C25, C26, C27, C28, C29, C3, C30, C4, C5, C6, C7, C8, C9: C, OH_Footprints:C_0603_1608Metric, symbol Device:C
- removed D1, D10, D11, D12, D13, D14, D15, D16, D17, D18, D19, D2, D20, D21, D22, D23, D24, D25, D26, D27, D28, D29, D3, D30, D31, D32, D33, D34, D35, D4, D5, D6, D7, D8, D9: WS2812B, OH_Footprints:LED_WS2812B_PLCC4_5.0x5.0mm_P3.2mm, symbol LED:WS2812B
- removed D36: LED, OH_Footprints:LED_D3.0mm, symbol Device:LED
- removed H1, H2: OHPanelScrew, OH_Footprints:OH_Panel_6-32_PHS, symbol KiCadCustomLib:OHPanelScrew
- removed J1, J2: Conn_01x04_Female, OH_Footprints:Molex_Mini-Fit_Jr_5566-04A_2x02_P4.20mm_Vertical, symbol Connector:Conn_01x04_Female
- removed LOGO1, LOGO2: OH_S2AL_Silkscreen, OH_Footprints:S3AL_Toggle_Silkscreen, symbol KiCadCustomLib:OH_S2AL_Silkscreen
- removed LOGO3, LOGO4: OH_S3AL_Silkscreen, OH_Footprints:S3AL_Toggle_Silkscreen, symbol KiCadCustomLib:OH_S3AL_Silkscreen
- removed LOGO5: OpenHornetLogoSmall, OH_Footprints:OH_LOGO_37.7mm_5.9mm, symbol KiCadCustomLib:OpenHornetLogoSmall
- removed LOGO6: CC-BY-NC-SA_Icon, OH_Footprints:CC-BY-NC-SA-Small, symbol KiCadCustomLib:CC-BY-NC-SA_Icon
- removed R1: R, OH_Footprints:R_0603_1608Metric, symbol Device:R
- added C1: 1000uF, OH_Footprints:CP_Elec_8x10, symbol OH_Symbols:Capacitor_Polarized_8x10_1000uF
- added C10, C11, C12, C13, C14, C15, C16, C17, C18, C19, C2, C20, C21, C22, C23, C24, C25, C26, C27, C28, C29, C3, C30, C4, C5, C6, C7, C8, C9: 0.1uF, OH_Footprints:C_0603_1608Metric, symbol OH_Symbols:Capacitor_0603_0.1uF
- added D1: Green, OH_Footprints:LED_D3.0mm, symbol OH_Symbols:LED_3.0mm_Green
- added D10, D11, D12, D13, D14, D15, D16, D17, D18, D19, D2, D20, D21, D22, D23, D24, D25, D26, D27, D28, D29, D3, D30, D31, D32, D33, D34, D35 (x2), D4, D5, D6, D7, D8, D9: WS2812B, OH_Footprints:LED_WS2812B_PLCC4_5.0x5.0mm_P3.2mm, symbol OH_Symbols:WS2812B
- added J1, J2: Mini-Fit Jr. 2x02, OH_Footprints:Molex_Mini-Fit_Jr_5566-04A_2x02_P4.20mm_Vertical, symbol OH_Symbols:Molex_Mini-Fit_Jr._2x02
- added LOGO1: LOGO, OH_Footprints:LOGO_OH_Text_Small, symbol OH_Symbols:LOGO_OpenHornet_Text_Small
- added LOGO2: LOGO, OH_Footprints:LOGO_CC-BY-NC-SA_Half_Small, symbol OH_Symbols:LOGO_License_Half_Small
- added MH1 (x2): 6x32 / 4mm, OH_Footprints:MountingHole_6-32_PHS, symbol OH_Symbols:MountingHole_6x32_PHS
- added MH10: Pot_B10K, OH_Footprints:BR10K_Pot_11mm_x_11mm, symbol OH_Symbols:MountingHole_B10K_Potentiometer
- added MH3, MH4, MH5, MH6: Switch_100SPx, OH_Footprints:100SPX_Toggle_13mm_x_18mm, symbol OH_Symbols:MountingHole_100SPx_Toggle
- added R1: 470, OH_Footprints:R_0603_1608Metric, symbol OH_Symbols:Resistor_0603_470Ω
- added TP1, TP2, TP3, TP4: TestPoint, OH_Footprints:TestPoint_THTPad_D1.5mm_Drill0.7mm, symbol OH_Symbols:TestPoint
Connections:
- new net: D10.2 (DOUT), D11.4 (DIN)
- new net: D10.4 (DIN), D9.2 (DOUT)
- new net: D13.2 (DOUT), D14.4 (DIN)
- new net: D34.2 (DOUT), D35.4 (DIN)
- new net: D33.2 (DOUT), D34.4 (DIN)
- new net: D35.2 (DOUT), D35.4 (DIN)
- new net: D28.2 (DOUT), D29.4 (DIN)
- new net: D25.2 (DOUT), D26.4 (DIN)
- new net: D24.2 (DOUT), D25.4 (DIN)
- new net: D8.2 (DOUT), D9.4 (DIN)
- new net: D22.2 (DOUT), D23.4 (DIN)
- new net: D21.2 (DOUT), D22.4 (DIN)
- new net: D4.2 (DOUT), D5.4 (DIN)
- new net: D3.2 (DOUT), D4.4 (DIN)
- new net: D19.2 (DOUT), D20.4 (DIN)
- new net: D18.2 (DOUT), D19.4 (DIN)
- new net: D26.2 (DOUT), D27.4 (DIN)
- new net: D17.2 (DOUT), D18.4 (DIN)
- new net: D16.2 (DOUT), D17.4 (DIN)
- new net: D32.2 (DOUT), D33.4 (DIN)
- new net: D31.2 (DOUT), D32.4 (DIN)
- new net: D12.2 (DOUT), D13.4 (DIN)
- new net: D11.2 (DOUT), D12.4 (DIN)
- new net: D1.1 (K), R1.1
- new net: D2.2 (DOUT), D3.4 (DIN)
- new net: D20.2 (DOUT), D21.4 (DIN)
- new net: D5.2 (DOUT), D6.4 (DIN)
- new net: D15.2 (DOUT), D16.4 (DIN)
- new net: D23.2 (DOUT), D24.4 (DIN)
- new net: D7.2 (DOUT), D8.4 (DIN)
- new net: D6.2 (DOUT), D7.4 (DIN)
- new net: D30.2 (DOUT), D31.4 (DIN)
- new net: D29.2 (DOUT), D30.4 (DIN)
- new net +5V: C1.1, C10.1, C11.1, C12.1, C13.1, C14.1, C15.1, C16.1, C17.1, C18.1, C19.1, C2.1, C20.1, C21.1, C22.1, C23.1, C24.1, C25.1, C26.1, C27.1, C28.1, C29.1, C3.1, C30.1, C4.1, C5.1, C6.1, C7.1, C8.1, C9.1, D1.2 (A), D10.1 (VDD), D11.1 (VDD), D12.1 (VDD), D13.1 (VDD), D14.1 (VDD), D15.1 (VDD), D16.1 (VDD), D17.1 (VDD), D18.1 (VDD), D19.1 (VDD), D2.1 (VDD), D20.1 (VDD), D21.1 (VDD), D22.1 (VDD), D23.1 (VDD), D24.1 (VDD), D25.1 (VDD), D26.1 (VDD), D27.1 (VDD), D28.1 (VDD), D29.1 (VDD), D3.1 (VDD), D30.1 (VDD), D31.1 (VDD), D32.1 (VDD), D33.1 (VDD), D34.1 (VDD), D35.1 (VDD), D35.1 (VDD), D4.1 (VDD), D5.1 (VDD), D6.1 (VDD), D7.1 (VDD), D8.1 (VDD), D9.1 (VDD), J1.1 (Pin_1), J1.2 (Pin_3), J2.1 (Pin_1), J2.2 (Pin_3), TP1.1
- new net DATA IN: D2.4 (DIN), J1.4 (Pin_4), TP3.1
- new net DATA OUT: D35.2 (DOUT), J2.4 (Pin_4), TP4.1
- new net DATA1: D14.2 (DOUT), D15.4 (DIN)
- new net DATA2: D27.2 (DOUT), D28.4 (DIN)
- new net GND: C1.2, C10.2, C11.2, C12.2, C13.2, C14.2, C15.2, C16.2, C17.2, C18.2, C19.2, C2.2, C20.2, C21.2, C22.2, C23.2, C24.2, C25.2, C26.2, C27.2, C28.2, C29.2, C3.2, C30.2, C4.2, C5.2, C6.2, C7.2, C8.2, C9.2, D10.3 (VSS), D11.3 (VSS), D12.3 (VSS), D13.3 (VSS), D14.3 (VSS), D15.3 (VSS), D16.3 (VSS), D17.3 (VSS), D18.3 (VSS), D19.3 (VSS), D2.3 (VSS), D20.3 (VSS), D21.3 (VSS), D22.3 (VSS), D23.3 (VSS), D24.3 (VSS), D25.3 (VSS), D26.3 (VSS), D27.3 (VSS), D28.3 (VSS), D29.3 (VSS), D3.3 (VSS), D30.3 (VSS), D31.3 (VSS), D32.3 (VSS), D33.3 (VSS), D34.3 (VSS), D35.3 (VSS), D35.3 (VSS), D4.3 (VSS), D5.3 (VSS), D6.3 (VSS), D7.3 (VSS), D8.3 (VSS), D9.3 (VSS), J1.3 (Pin_2), J2.3 (Pin_2), R1.2, TP2.1
Other:
- company: (none) -> www.openhornet.com
